File: TooManyKeys/TooManyKeys.sch (KiCad schematic (older format))
At the start: 59 parts

Commit message: V1 Schematics
Connections:
- net SW8: now reaches MASTER_U?.10 (SW8)
- net SW9: now reaches MASTER_U?.11 (SW9)
- net SW10: now reaches MASTER_U?.13 (SW10)
- net SW11: now reaches MASTER_U?.14 (SW11)
- net SW12: now reaches MASTER_U?.15 (SW12)
- net CS1: now reaches MASTER_U?.16 (CS1)
- net CS2: now reaches MASTER_U?.17 (CS2)
- net CS3: now reaches MASTER_U?.18 (CS3)
- net CS4: now reaches MASTER_U?.19 (CS4)
- net SW1: now reaches MASTER_U?.2 (SW1)
- net CS5: now reaches MASTER_U?.21 (CS5)
- net CS6: now reaches MASTER_U?.22 (CS6)
- net CS7: now reaches MASTER_U?.23 (CS7)
- net CS8: now reaches MASTER_U?.24 (CS8)
- net CS9: now reaches MASTER_U?.25 (CS9)
- net CS10: now reaches MASTER_U?.26 (CS10)
- net CS11: now reaches MASTER_U?.27 (CS11)
- net CS12: now reaches MASTER_U?.28 (CS12)
- net SW2: now reaches MASTER_U?.3 (SW2)
- net CS13: now reaches MASTER_U?.30 (CS13)
- net CS14: now reaches MASTER_U?.31 (CS14)
- net CS15: now reaches MASTER_U?.32 (CS15)
- net CS16: now reaches MASTER_U?.33 (CS16)
- net SW3: now reaches MASTER_U?.4 (SW3)
- net SW4: now reaches MASTER_U?.6 (SW4)
- net SW5: now reaches MASTER_U?.7 (SW5)
- net SW6: now reaches MASTER_U?.8 (SW6)
- net SW7: now reaches MASTER_U?.9 (SW7)
- net SW20: now reaches SLAVE_U?.10 (SW8)
- net SW21: now reaches SLAVE_U?.11 (SW9)
- net SW22: now reaches SLAVE_U?.13 (SW10)
- net SW23: now reaches SLAVE_U?.14 (SW11)
- net SW24: now reaches SLAVE_U?.15 (SW12)
- net CS17: now reaches SLAVE_U?.16 (CS1)
- net CS18: now reaches SLAVE_U?.17 (CS2)
- net CS19: now reaches SLAVE_U?.18 (CS3)
- net CS20: now reaches SLAVE_U?.19 (CS4)
- net SW13: now reaches SLAVE_U?.2 (SW1)
- net CS21: now reaches SLAVE_U?.21 (CS5)
- net CS22: now reaches SLAVE_U?.22 (CS6)
- net CS23: now reaches SLAVE_U?.23 (CS7)
- net CS24: now reaches SLAVE_U?.24 (CS8)
- net CS25: now reaches SLAVE_U?.25 (CS9)
- net CS26: now reaches SLAVE_U?.26 (CS10)
- net CS27: now reaches SLAVE_U?.27 (CS11)
- net CS28: now reaches SLAVE_U?.28 (CS12)
- net SW14: now reaches SLAVE_U?.3 (SW2)
- net SW15: now reaches SLAVE_U?.4 (SW3)
- net SW16: now reaches SLAVE_U?.6 (SW4)
- net SW17: now reaches SLAVE_U?.7 (SW5)
- net SW18: now reaches SLAVE_U?.8 (SW6)
- net SW19: now reaches SLAVE_U?.9 (SW7)
Changed lines of the file:
@@
 Wire Wire Line
 	12550 5800 13200 5800
+Text GLabel 11150 8550 2    50   Input ~ 0
+SW1
+Text GLabel 11150 8650 2    50   Input ~ 0
+SW2
+Text GLabel 11150 8750 2    50   Input ~ 0
+SW3
+Text GLabel 11150 8850 2    50   Input ~ 0
+SW4
+Text GLabel 11150 8950 2    50   Input ~ 0
+SW5
+Text GLabel 11150 9050 2    50   Input ~ 0
+SW6
+Text GLabel 11150 9150 2    50   Input ~ 0
+SW7
+Text GLabel 11150 9250 2    50   Input ~ 0
+SW8
+Text GLabel 11150 9350 2    50   Input ~ 0
+SW9
+Text GLabel 11150 9450 2    50   Input ~ 0
+SW10
+Text GLabel 11150 9550 2    50   Input ~ 0
+SW11
+Text GLabel 11150 9650 2    50   Input ~ 0
+SW12
+Text GLabel 15250 7000 2    50   Input ~ 0
+SW13
+Text GLabel 15250 7100 2    50   Input ~ 0
+SW14
+Text GLabel 15250 7200 2    50   Input ~ 0
+SW15
+Text GLabel 15250 7300 2    50   Input ~ 0
+SW16
+Text GLabel 15250 7400 2    50   Input ~ 0
+SW17
+Text GLabel 15250 7500 2    50   Input ~ 0
+SW18
+Text GLabel 15250 7600 2    50   Input ~ 0
+SW19
+Text GLabel 15250 7700 2    50   Input ~ 0
+SW20
+Text GLabel 15250 7800 2    50   Input ~ 0
+SW21
+Text GLabel 15250 7900 2    50   Input ~ 0
+SW22
+Text GLabel 15250 8000 2    50   Input ~ 0
+SW23
+Text GLabel 15250 8100 2    50   Input ~ 0
+SW24
+Text GLabel 11150 6850 2    50   Input ~ 0
+CS1
+Text GLabel 11150 6950 2    50   Input ~ 0
+CS2
+Text GLabel 11150 7050 2    50   Input ~ 0
+CS3
+Text GLabel 11150 7150 2    50   Input ~ 0
+CS4
+Text GLabel 11150 7250 2    50   Input ~ 0
+CS5
+Text GLabel 11150 7350 2    50   Input ~ 0
+CS6
+Text GLabel 11150 7450 2    50   Input ~ 0
+CS7
+Text GLabel 11150 7550 2    50   Input ~ 0
+CS8
+Text GLabel 11150 7650 2    50   Input ~ 0
+CS9
+Text GLabel 11150 7750 2    50   Input ~ 0
+CS10
+Text GLabel 11150 7850 2    50   Input ~ 0
+CS11
+Text GLabel 11150 7950 2    50   Input ~ 0
+CS12
+Text GLabel 11150 8050 2    50   Input ~ 0
+CS13
+Text GLabel 11150 8150 2    50   Input ~ 0
+CS14
+Text GLabel 11150 8250 2    50   Input ~ 0
+CS15
+Text GLabel 11150 8350 2    50   Input ~ 0
+CS16
+Text GLabel 15250 5300 2    50   Input ~ 0
+CS17
+Text GLabel 15250 5400 2    50   Input ~ 0
+CS18
+Text GLabel 15250 5500 2    50   Input ~ 0
+CS19
+Text GLabel 15250 5600 2    50   Input ~ 0
+CS20
+Text GLabel 15250 5700 2    50   Input ~ 0
+CS21
+Text GLabel 15250 5800 2    50   Input ~ 0
+CS22
+Text GLabel 15250 5900 2    50   Input ~ 0
+CS23
+Text GLabel 15250 6000 2    50   Input ~ 0
+CS24
+Text GLabel 15250 6100 2    50   Input ~ 0
+CS25
+Text GLabel 15250 6200 2    50   Input ~ 0
+CS26
+Text GLabel 15250 6300 2    50   Input ~ 0
+CS27
+Text GLabel 15250 6400 2    50   Input ~ 0
+CS28
 $EndSCHEMATC

Commit message: WIP pcb
Parts:
- C1, C10, C11, C12, C2, C3, C8, C9: renamed from C?; footprint Capacitors_SMD:C_0603 -> Capacitor_SMD:C_0805_2012Metric
- C13, C14, C15, C16, C17, C18, C19, C20, C21, C22, C23, C24, C25, C26, C27, C28, C29, C30, C4, C5, C6, C7: renamed from C?; footprint (none) -> Capacitor_SMD:C_0805_2012Metric
- F1: renamed from F?; footprint (none) -> Fuse:Fuse_1206_3216Metric
- J1: renamed from J?; footprint 5051103091 -> SamacSys_Parts:0541043033
- MASTER_U1: renamed from MASTER_U?; footprint Package_QFP:TQFP-48-1EP_7x7mm_P0.5mm_EP5x5mm -> SamacSys_Parts:QFP50P900X900X120-49N
- R1, R10, R11, R12, R13, R14, R15, R16, R17, R18, R2, R3, R4, R5, R6, R7, R8, R9: renamed from R?; footprint (none) -> Resistor_SMD:R_0805_2012Metric
- SLAVE_U1: renamed from SLAVE_U?; footprint Package_QFP:TQFP-48-1EP_7x7mm_P0.5mm_EP5x5mm -> SamacSys_Parts:QFP50P900X900X120-49N
- SW1: renamed from SW?; footprint (none) -> random-keyboard-parts:SKQG-1155865
- U1: renamed from U?; footprint (none) -> random-keyboard-parts:SOT143B
- U2: renamed from U?; footprint Package_QFP:TQFP-64_14x14mm_P0.8mm -> SamacSys_Parts:QFP80P1600X1600X120-64N
- U3: renamed from U?; footprint (none) -> SamacSys_Parts:SOP50P310X90-8N
- USB1: renamed from USB?; footprint (none) -> Type-C:HRO-TYPE-C-31-M-12
- Y1: renamed from Y?; footprint (none) -> Crystal:Crystal_SMD_3225-4Pin_3.2x2.5mm
- gave numbers to parts that had none: 1

Commit message: changes made to schematics following upwork
Parts:
- MASTER_U1, SLAVE_U1: value IS31FL3733-TQ -> IS31FL3733-QFLS4-TR; footprint SamacSys_Parts:QFP50P900X900X120-49N -> SamacSys_Parts:QFN40P600X600X80-49N-D
Connections:
- net SYNC: now reaches MASTER_U1.40 (SYNC)
- net SYNC: now also SLAVE_U1.40 (SYNC)
Other:
- moved on the sheet: R15, R18, R5, R6

Commit message: Final Schematic version, starting work on pcb
Parts:
- added J2: AVR-ISP-6(SWR204-NRTN-D03-RA-GA), SamacSys_Parts:SWR204NRTND03STGA, symbol Connector:AVR-ISP-6
- F1: value 500mA -> 1A
- J1: symbol SamacSys_Parts:505110-3091_Oled -> TooManyKeys-rescue:505110-3091_Oled-SamacSys_Parts
- MASTER_U1, SLAVE_U1: value IS31FL3733-QFLS4-TR -> IS31FL3733-TQ; footprint SamacSys_Parts:QFN40P600X600X80-49N-D -> SamacSys_Parts:QFP50P900X900X120-49N
- U1: symbol random-keyboard-parts:PRTR5V0U2X -> TooManyKeys-rescue:PRTR5V0U2X-random-keyboard-parts
- U4: value AP1117-33 -> AZ1117CH-3.3TRG1
- USB1: symbol Type-C:HRO-TYPE-C-31-M-12 -> TooManyKeys-rescue:HRO-TYPE-C-31-M-12-Type-C
Connections:
- net +5V: now also C13.2, C14.2, C16.2, C17.2, C20.2, C21.2, J2.2 (VCC); no longer C13.1, C14.1, C16.1, C17.1, C20.1, C21.1
- net GND: now also C13.1, C14.1, C16.1, C17.1, C20.1, C21.1, J2.6 (GND); no longer C13.2, C14.2, C16.2, C17.2, C20.2, C21.2
- net RESET: now also J2.5 (~RST)
- net ROW0: now also U2.51 (PA0); no longer U2.10 (PB0)
- net ROW1: now also U2.50 (PA1); no longer U2.11 (PB1)
- net ROW2: now also U2.49 (PA2); no longer U2.12 (PB2)
- net ROW3: now also U2.48 (PA3); no longer U2.13 (PB3)
- net ROW4: now also U2.47 (PA4); no longer U2.14 (PB4)
- net ROW5: now also U2.46 (PA5); no longer U2.15 (PB5)
- net ROW6: now also U2.45 (PA6); no longer U2.16 (PB6)
- net ROW7: now also U2.44 (PA7); no longer U2.17 (PB7)
- net SCL_3.3: now also R6.1; no longer R5.2
- net SDA_3.3: now also R5.2; no longer R6.1
- net COL23: no longer names the net of U2.57 (PF4)
- new net MISO: J2.1 (MISO), U2.13 (PB3)
- new net MOSI: J2.4 (MOSI), U2.12 (PB2)
- new net SCK: J2.3 (SCK), U2.11 (PB1)
Other:
- moved on the sheet: C1, C12, C13, C14, C16, C17, C2, C20, C21, C3, C4, C6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
