File: TooManyKeys/TooManyKeys.kicad_pcb (KiCad board)
At the start: 2 copper layers, 392 parts, among them J1 54104-3031_Oled, SW1 SW_Push, U1 PRTR5V0U2X, U2 AT90USB1286-AU, U3 PCA9306, U4 AP1117-33, Y1 16MHz

Commit message: WIP pcb 2
Parts:
- D1, D10, D11, D12, D13, D14, D15, D16, D17, D18, D19, D2, D20, D21, D22, D23, D24, D25, D26, D27, D28, D29, D3, D30, D31, D32, D33, D34, D35, D36, D37, D38, D39, D4, D40, D41, D42, D43, D44, D45, D46, D47, D48, D49, D5, D50, D51, D52, D53, D54, D55, D56, D57, D58, D59, D6, D60, D61, D62, D63, D68, D7, D8, D9: moved to B.Cu
- MX_P+1, MX_PENT1: footprint MX_Only:MXOnly-2U-NoLED -> MX_Only:MXOnly-2U-NoLED_Vertical
- MX_RCTL1: footprint MX_Only:MXOnly-1U-NoLED -> MX_Only:MXOnly-1.25U-NoLED
- MX_RGHT1: footprint MX_Only:MXOnly-1.25U-NoLED -> MX_Only:MXOnly-1U-NoLED
- moved MX_PENT1 688.9 mm to (585.8, 368.3)
- moved MX_P0 659.1 mm to (538.2, 377.8)
- moved MX_P+1 646.1 mm to (585.8, 330.2)
- moved MX_P/1 612.2 mm to (547.7, 301.6)
- moved MX_P-1 595.1 mm to (585.8, 301.6)
- moved MX_P2 585.9 mm to (547.7, 358.8)
- moved MX_RGHT1 585.9 mm to (504.8, 377.8)
- moved MX_P3 584.8 mm to (566.7, 358.8)
- moved MX_PDOT1 578.6 mm to (566.7, 377.8)
- moved MX_UP1 571.5 mm to (485.8, 358.8)
- moved D44 565.9 mm to (593.7, 301.6), turned to 90 degrees
- moved D7 560.2 mm to (512.8, 258.8), turned to 90 degrees
- moved MX_RSFT1 557.5 mm to (426.2, 358.8)
- moved D43 552.7 mm to (574.7, 301.6), turned to 90 degrees
- moved D6 552.4 mm to (493.7, 258.8), turned to 90 degrees
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
Commit message: changes made to schematics following upwork
Parts:
- C1, C10, C11, C12, C13, C14, C15, C16, C17, C18, C19, C2, C20, C21, C22, C23, C24, C25, C26, C27, C28, C29, C3, C30, C4, C5, C6, C7, C8, C9, D100, D101, D102, D103, D104, D105, D106, D107, D108, D109, D110, D111, D64, D65, D66, D67, D69, D70, D71, D72, D73, D74, D75, D76, D77, D78, D79, D80, D81, D82, D83, D84, D85, D86, D87, D88, D89, D90, D91, D92, D93, D94, D95, D96, D97, D98, D99, F1, J1, LED1, LED10, LED100, LED101, LED102, LED103, LED104, LED105, LED106, LED107, LED108, LED109, LED11, LED110, LED111, LED12, LED13, LED14, LED15, LED16, LED17, LED18, LED19, LED2, LED20, LED21, LED22, LED23, LED24, LED25, LED26, LED27, LED28, LED29, LED3, LED30, LED31, LED32, LED33, LED34, LED35, LED36, LED37, LED38, LED39, LED4, LED40, LED41, LED42, LED43, LED44, LED45, LED46, LED47, LED48, LED49, LED5, LED50, LED51, LED52, LED53, LED54, LED55, LED56, LED57, LED58, LED59, LED6, LED60, LED61, LED62, LED63, LED64, LED65, LED66, LED67, LED68, LED69, LED7, LED70, LED71, LED72, LED73, LED74, LED75, LED76, LED77, LED78, LED79, LED8, LED80, LED81, LED82, LED83, LED84, LED85, LED86, LED87, LED88, LED89, LED9, LED90, LED91, LED92, LED93, LED94, LED95, LED96, LED97, LED98, LED99, R1, R10, R11, R12, R13, R14, R15, R16, R17, R18, R2, R3, R4, R5, R6, R7, R8, R9, SW1, U1, U2, U3, U4, USB1, Y1: moved to B.Cu
- MASTER_U1, SLAVE_U1: value IS31FL3733-TQ -> IS31FL3733-QFLS4-TR; moved to B.Cu
- moved LED101 619.4 mm to (566.7, 326.2)
- moved LED97 609.1 mm to (547.7, 307.2)
- moved LED98 607.4 mm to (566.7, 307.2)
- moved LED102 604.2 mm to (585.8, 335.8)
- moved LED16 598.7 mm to (528.6, 326.2)
- moved LED99 590.6 mm to (585.8, 307.2)
- moved LED61 587.2 mm to (566.7, 383.4)
- moved LED100 582.3 mm to (547.7, 326.2)
- moved LED46 576.5 mm to (585.8, 373.9)
- moved LED29 576.1 mm to (547.7, 345.3)
- moved LED45 572.7 mm to (566.7, 364.3)
- moved LED28 568.6 mm to (528.6, 345.3)
- moved LED30 549.8 mm to (566.7, 345.3)
- moved LED60 543.6 mm to (538.2, 383.4)
- moved LED95 536.8 mm to (504.8, 307.2)
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Routing:
- net GND: track 0.00 -> 54.2 mm
- net Net-(D1-Pad1): track 0.00 -> 19.6 mm
- net VCC: track 0.00 -> 7.03 mm
- net Net-(D42-Pad2): track 0.00 -> 6.82 mm
- net Net-(D5-Pad2): track 0.00 -> 6.82 mm
- net Net-(D38-Pad2): track 0.00 -> 6.82 mm
- net Net-(D33-Pad2): track 0.00 -> 6.82 mm
- net Net-(D32-Pad2): track 0.00 -> 6.82 mm
- net Net-(D3-Pad2): track 0.00 -> 6.82 mm
- net Net-(D28-Pad2): track 0.00 -> 6.82 mm
- net Net-(D21-Pad2): track 0.00 -> 6.82 mm
- net Net-(D20-Pad2): track 0.00 -> 6.82 mm
- net Net-(D19-Pad2): track 0.00 -> 6.82 mm
- net Net-(D13-Pad2): track 0.00 -> 6.82 mm
- net Net-(D11-Pad2): track 0.00 -> 6.82 mm
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- added copper zone on B.Cu, net GND
- added copper zone on F.Cu, net GND
Other:
- board outline added: 430.2 x 139.7 mm
- net class Default: trace_width 0.25 -> 0.254
- net class Power added: clearance 0.2, trace_width 0.381, via_dia 0.8, via_drill 0.4

Commit message: Final Schematic version, starting work on pcb
Parts:
- added J2: AVR-ISP-6(SWR204-NRTN-D03-RA-GA), SamacSys_Parts:SWR204NRTND03STGA, B.Cu at (445.3, 251.2)
- F1: value 500mA -> 1A
- MASTER_U1, SLAVE_U1: value IS31FL3733-QFLS4-TR -> IS31FL3733-TQ
- U4: value AP1117-33 -> AZ1117CH-3.3TRG1
- moved F1 161.5 mm to (361.2, 251.2), turned to 0 degrees
- moved R8 54.4 mm to (527.8, 254.3), turned to 90 degrees
- moved C4 46.1 mm to (542.8, 251.7)
- moved C10 44.6 mm to (532.4, 254.3), turned to 270 degrees
- moved C3 43.6 mm to (538.7, 251.7), turned to 180 degrees
- moved C11 41.7 mm to (537.0, 258.0)
- moved C8 38.8 mm to (527.8, 258.0)
- moved C9 38.8 mm to (532.4, 258.1)
- moved R9 28.6 mm to (547.3, 251.7), turned to 180 degrees
- moved C12 24.9 mm to (555.8, 251.6), turned to 180 degrees
- moved C6 23.5 mm to (551.7, 251.7), turned to 0 degrees
- moved R6 21.2 mm to (563.8, 251.6), turned to 0 degrees
- moved C7 20.2 mm to (559.8, 251.6), turned to 180 degrees
- moved C1 19.5 mm to (571.6, 251.7), turned to 0 degrees
- moved R1 18.6 mm to (544.6, 261.6), turned to 270 degrees
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Connections:
- net COL23 renamed Net-(U2-Pad57)
- C13 pad 1: +5V -> GND
- C13 pad 2: GND -> +5V
- C14 pad 1: +5V -> GND
- C14 pad 2: GND -> +5V
- C16 pad 1: +5V -> GND
- C16 pad 2: GND -> +5V
- C17 pad 1: +5V -> GND
- C17 pad 2: GND -> +5V
- C20 pad 1: +5V -> GND
- C20 pad 2: GND -> +5V
- C21 pad 1: +5V -> GND
- C21 pad 2: GND -> +5V
- D1 pad 1: Net-(D1-Pad1) -> ROW0
- D2 pad 1: Net-(D1-Pad1) -> ROW0
- D3 pad 1: Net-(D1-Pad1) -> ROW0
- D4 pad 1: Net-(D1-Pad1) -> ROW0
- D5 pad 1: Net-(D1-Pad1) -> ROW0
- D6 pad 1: Net-(D1-Pad1) -> ROW0
- D7 pad 1: Net-(D1-Pad1) -> ROW0
- MASTER_U1 pad 40: Net-(MASTER_U1-Pad40) -> SYNC
- R5 pad 2: SCL_3.3 -> SDA_3.3
- R6 pad 1: SDA_3.3 -> SCL_3.3
- SLAVE_U1 pad 40: Net-(SLAVE_U1-Pad40) -> SYNC
- U2 pad 10: ROW0 -> Net-(U2-Pad10)
- U2 pad 11: ROW1 -> SCK
- U2 pad 12: ROW2 -> MOSI
- U2 pad 13: ROW3 -> MISO
- U2 pad 14: ROW4 -> Net-(U2-Pad14)
- U2 pad 15: ROW5 -> Net-(U2-Pad15)
- U2 pad 16: ROW6 -> Net-(U2-Pad16)
- U2 pad 17: ROW7 -> Net-(U2-Pad17)
- U2 pad 44: Net-(U2-Pad44) -> ROW7
- U2 pad 45: Net-(U2-Pad45) -> ROW6
- U2 pad 46: Net-(U2-Pad46) -> ROW5
- U2 pad 47: Net-(U2-Pad47) -> ROW4
- U2 pad 48: Net-(U2-Pad48) -> ROW3
- U2 pad 49: Net-(U2-Pad49) -> ROW2
- U2 pad 50: Net-(U2-Pad50) -> ROW1
- U2 pad 51: Net-(U2-Pad51) -> ROW0
Routing:
- net GND: track 54.2 -> 2.09 mm
- net Net-(D1-Pad1): track 19.6 -> 0.00 mm
- net Net-(D97-Pad2): track 0.00 -> 8.84 mm
- net Net-(D64-Pad2): track 0.00 -> 8.84 mm
- net VCC: track 7.03 -> 0.00 mm
- net Net-(D96-Pad2): track 0.00 -> 6.82 mm
- net Net-(D80-Pad2): track 0.00 -> 6.82 mm
- net Net-(D91-Pad2): track 0.00 -> 6.82 mm
- net Net-(D90-Pad2): track 0.00 -> 6.82 mm
- net Net-(D86-Pad2): track 0.00 -> 6.82 mm
- net Net-(D85-Pad2): track 0.00 -> 6.82 mm
- net Net-(D78-Pad2): track 0.00 -> 6.82 mm
- net Net-(D73-Pad2): track 0.00 -> 6.82 mm
- net Net-(D72-Pad2): track 0.00 -> 6.82 mm
- net Net-(D107-Pad2): track 0.00 -> 6.82 mm
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
Commit message: V1 New Led Positions
Parts:
- removed LED50: XZMDKCBDDG45S-9, SamacSys_Parts:XZMDKCBDDG45S9
- added LEDe: XZMDKCBDDG45S-9, SamacSys_Parts:XZMDKCBDDG45S9, B.Cu at (188.1, 364.3)
- moved LED46 369.1 mm to (233.4, 264.3)
- moved LED69 357.7 mm to (566.7, 326.1)
- moved LED45 343.1 mm to (233.4, 283.4)
- moved LED70 343.0 mm to (566.7, 345.2)
- moved LED71 329.8 mm to (566.7, 364.2)
- moved LED61 329.2 mm to (238.1, 364.3)
- moved LED44 319.5 mm to (233.4, 307.2)
- moved LED72 318.3 mm to (566.7, 383.3)
- moved LED60 312.0 mm to (226.2, 383.3)
- moved LED76 310.2 mm to (485.8, 264.3)
- moved LED59 302.4 mm to (202.4, 383.4)
- moved LED77 291.1 mm to (504.8, 264.3)
- moved LED43 288.3 mm to (242.9, 326.2)
- moved LED78 271.5 mm to (504.8, 283.4)
- moved LED58 267.4 mm to (219.1, 364.3)
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Routing:
- net D+: track 0.00 -> 170.1 mm
- net D-: track 0.00 -> 170.1 mm
- net GND: track 2.09 -> 4.86 mm

Commit message: Led alignment
Parts:
- moved LED65 0.26 mm to (585.8, 373.9)
- moved LED83 0.11 mm to (528.6, 364.3)
- moved LED84 0.11 mm to (528.6, 345.3)
- moved LED66 0.11 mm to (585.8, 335.8)
- moved LED70 0.11 mm to (566.7, 345.3)
- moved LED71 0.11 mm to (566.7, 364.3)
- moved LED72 0.11 mm to (566.7, 383.4)
- moved LED73 0.11 mm to (547.7, 364.3)
- moved LED74 0.11 mm to (547.7, 345.3)
- moved LED82 0.11 mm to (538.2, 383.4)
- moved LED4 0.11 mm to (376.2, 326.2)
- moved LED101 0.11 mm to (395.3, 326.2)
- moved LED107 0.11 mm to (414.3, 326.2)
- moved LED69 0.11 mm to (566.7, 326.2)
- moved LED75 0.11 mm to (547.7, 326.2)
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Routing:
- net Net-(R2-Pad2): track 0.03 -> 11.5 mm
- net Net-(R3-Pad2): track 0.00 -> 11.2 mm
- net Net-(D77-Pad2): track 0.00 -> 6.82 mm
- net Net-(D76-Pad2): track 0.00 -> 6.82 mm

Commit message: Partial Routing
Routing:
- net ROW6: track 0.00 -> 832.6 mm, vias 0 -> 4
- net ROW5: track 0.00 -> 759.9 mm, vias 0 -> 7
- net ROW4: track 0.00 -> 707.5 mm, vias 0 -> 2
- net ROW3: track 0.00 -> 701.6 mm, vias 0 -> 2
- net SW2: track 0.00 -> 699.8 mm, vias 0 -> 11
- net SW9: track 0.00 -> 636.7 mm, vias 0 -> 20
- net SW3: track 0.00 -> 632.4 mm, vias 0 -> 18
- net SW1: track 0.00 -> 617.1 mm, vias 0 -> 22
- net COL02: track 0.00 -> 595.4 mm, vias 0 -> 4
- net +5V: track 0.00 -> 583.4 mm, vias 0 -> 8
- net ROW1: track 0.00 -> 581.8 mm
- net SW23: track 0.00 -> 577.9 mm, vias 0 -> 20
- net SW22: track 0.00 -> 563.1 mm, vias 0 -> 12
- net COL04: track 0.00 -> 559.6 mm, vias 0 -> 4
- net CS8: track 0.00 -> 546.8 mm, vias 0 -> 9
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