File: TooManyKeys/TooManyKeys.kicad_pcb (KiCad board)
At the start: 2 copper layers, 430.2 x 139.7 mm, 393 parts, among them J1 54104-3031_Oled, J2 AVR-ISP-6(SWR204-NRTN-D03-RA-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, SW1 SW_Push, U1 PRTR5V0U2X, U2 AT90USB1286-AU, U3 PCA9306, U4 AZ1117CH-3.3TRG1, Y1 16MHz

Commit message: New footprint, pcb key matrix completed
Parts:
- added G***: LOGO, bitmap:Logo, B.Cu at (483.4, 339.7)
- MX_0, MX_1, MX_2, MX_3, MX_4, MX_5, MX_6, MX_7, MX_8, MX_9, MX_A1, MX_B1, MX_C1, MX_COMM1, MX_D1, MX_DEL1, MX_DOT1, MX_DOWN1, MX_E1, MX_END1, MX_EQL1, MX_ESC1, MX_F1, MX_F10, MX_F11, MX_F12, MX_F13, MX_F2, MX_F3, MX_F4, MX_F5, MX_F6, MX_F7, MX_F8, MX_F9, MX_G1, MX_GRV1, MX_H1, MX_HOME1, MX_I1, MX_INS1, MX_J1, MX_K1, MX_L1, MX_LBRC1, MX_LEFT1, MX_M1, MX_MINS1, MX_MUTE1, MX_N1, MX_NEXT1, MX_NLCK1, MX_O1, MX_P*1, MX_P-1, MX_P/1, MX_P1, MX_P10, MX_P2, MX_P3, MX_P4, MX_P5, MX_P6, MX_P7, MX_P8, MX_P9, MX_PAUSE1, MX_PDOT1, MX_PGDN1, MX_PGUP1, MX_PLAY1, MX_PREV1, MX_PSCR1, MX_Q1, MX_QUOT1, MX_R1, MX_RBRC1, MX_RGHT1, MX_S1, MX_SCLN1, MX_SLCK1, MX_SLSH1, MX_STOP1, MX_T1, MX_U1, MX_UP1, MX_V1, MX_VOLD1, MX_VOLU1, MX_W1, MX_X1, MX_Y1, MX_Z1: footprint MX_Only:MXOnly-1U-NoLED -> MX_Only:MXOnly-1U-NoLED_3Pins
- MX_BSLS1, MX_TAB1: footprint MX_Only:MXOnly-1.5U-NoLED -> MX_Only:MXOnly-1.5U-NoLED_3Pins
- MX_BSPC1, MX_P0: footprint MX_Only:MXOnly-2U-NoLED -> MX_Only:MXOnly-2U-NoLED_3Pins
- MX_CAPS1: footprint MX_Only:MXOnly-1.75U-NoLED -> MX_Only:MXOnly-1.75U-NoLED_3Pins
- MX_ENT1, MX_LSFT1: footprint MX_Only:MXOnly-2.25U-NoLED -> MX_Only:MXOnly-2.25U-NoLED_3Pins
- MX_LALT1, MX_LCTL1, MX_LGUI1, MX_MENU1, MX_RALT1, MX_RCTL1, MX_RGUI1: footprint MX_Only:MXOnly-1.25U-NoLED -> MX_Only:MXOnly-1.25U-NoLED_3Pins
- MX_P+1, MX_PENT1: footprint MX_Only:MXOnly-2U-NoLED_Vertical -> MX_Only:MXOnly-2U-NoLED_3Pins
- MX_RSFT1: footprint MX_Only:MXOnly-2.75U-NoLED -> MX_Only:MXOnly-2.75U-NoLED_3Pins
- MX_SPC1: footprint MX_Only:MXOnly-6.25U-NoLED -> MX_Only:MXOnly-6.25U-NoLED_3Pins
- moved D98 11.5 mm to (585.7, 376.5), turned to 0 degrees
- moved D65 11.4 mm to (585.7, 338.3), turned to 0 degrees
- moved LED66 7.81 mm to (580.2, 330.3), turned to 270 degrees
- moved LED65 7.73 mm to (580.2, 368.6), turned to 270 degrees
- moved U1 2.38 mm to (371.5, 259.5)
- moved R2 2.38 mm to (369.1, 263.4)
- moved R3 2.38 mm to (373.9, 263.4)
- moved R14 0.39 mm to (388.7, 257.0)
- moved MX_PENT1 0.26 mm to (585.7, 368.6), turned to 270 degrees
- moved C14 0.25 mm to (427.9, 256.4)
- moved MX_P+1 0.14 mm to (585.7, 330.3), turned to 270 degrees
- moved C30 0.13 mm to (343.7, 256.3)
- moved R17 0.10 mm to (307.7, 255.8)
- turned Y1 to 135 degrees
- renumbered LEDe to LED50
Connections:
- U2 pad 18: COL15 -> Net-(U2-Pad18)
- U2 pad 19: COL16 -> Net-(U2-Pad19)
- U2 pad 2: COL18 -> COL14
- U2 pad 27: COL08 -> Net-(U2-Pad27)
- U2 pad 28: COL09 -> Net-(U2-Pad28)
- U2 pad 29: COL10 -> Net-(U2-Pad29)
- U2 pad 30: COL11 -> Net-(U2-Pad30)
- U2 pad 31: COL12 -> COL16
- U2 pad 32: COL13 -> COL15
- U2 pad 33: Net-(U2-Pad33) -> COL12
- U2 pad 34: Net-(U2-Pad34) -> COL13
- U2 pad 49: ROW2 -> ROW1
- U2 pad 50: ROW1 -> ROW0
- U2 pad 51: ROW0 -> Net-(U2-Pad51)
- U2 pad 54: Net-(U2-Pad54) -> COL22
- U2 pad 55: Net-(U2-Pad55) -> COL21
- U2 pad 56: Net-(U2-Pad56) -> COL20
- U2 pad 57: Net-(U2-Pad57) -> COL19
- U2 pad 58: COL22 -> COL08
- U2 pad 59: COL21 -> COL09
- U2 pad 60: COL20 -> COL10
- U2 pad 61: COL19 -> COL11
- U2 pad 9: COL14 -> Net-(U2-Pad9)
Routing:
- net SW2: track 699.8 -> 0.00 mm, vias 11 -> 0
- net SW9: track 636.7 -> 0.01 mm, vias 20 -> 0
- net SW3: track 632.4 -> 0.00 mm, vias 18 -> 0
- net SW1: track 617.1 -> 0.00 mm, vias 22 -> 0
- net +5V: track 583.4 -> 0.00 mm, vias 8 -> 0
- net SW23: track 577.9 -> 0.00 mm, vias 20 -> 0
- net SW22: track 563.1 -> 0.00 mm, vias 12 -> 0
- net CS8: track 546.8 -> 0.00 mm, vias 9 -> 0
- net CS4: track 516.4 -> 0.00 mm, vias 8 -> 0
- net SW8: track 510.6 -> 0.00 mm, vias 16 -> 0
- net SW18: track 507.4 -> 0.00 mm, vias 18 -> 0
- net CS7: track 499.3 -> 0.00 mm, vias 7 -> 0
- net SW12: track 498.2 -> 0.00 mm, vias 17 -> 0
- net SW7: track 497.5 -> 0.00 mm, vias 13 -> 0
- net SW16: track 479.3 -> 0.00 mm, vias 17 -> 0
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
Commit message: Before changing to new led and moving mcu caps and usb resistors
Parts:
- moved R2 151.7 mm to (520.8, 262.6), turned to 180 degrees
- moved R3 147.0 mm to (520.8, 260.6), turned to 180 degrees
- moved C28 34.6 mm to (340.4, 263.1), turned to 0 degrees
- moved R17 32.7 mm to (338.3, 267.2), turned to 0 degrees
- moved C27 31.4 mm to (322.1, 254.0)
- moved R8 30.4 mm to (530.9, 284.5), turned to 270 degrees
- moved R16 29.3 mm to (338.3, 265.2), turned to 0 degrees
- moved C19 28.8 mm to (417.6, 252.0)
- moved C17 28.5 mm to (408.9, 253.5), turned to 315 degrees
- moved R18 24.6 mm to (336.8, 256.0)
- moved C26 24.5 mm to (324.1, 254.0)
- moved C10 24.3 mm to (521.2, 275.8), turned to 0 degrees
- moved R14 21.3 mm to (408.4, 265.2), turned to 180 degrees
- moved R13 21.3 mm to (408.4, 267.2), turned to 180 degrees
- moved R15 17.8 mm to (410.5, 252.0), turned to 135 degrees
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Routing:
- net D-: track 168.3 -> 0.00 mm
- net D+: track 168.3 -> 0.00 mm
- net RESET: track 38.8 -> 0.00 mm
- net GND: track 32.2 -> 6.60 mm
- net SCL: track 9.60 -> 0.00 mm
- net SW16: track 0.00 -> 6.34 mm
- net SW15: track 0.00 -> 6.30 mm
- net Net-(R7-Pad2): track 7.64 -> 12.9 mm
- net SDA: track 4.43 -> 0.00 mm
- net Net-(R8-Pad1): track 0.00 -> 3.77 mm
- net ROW7: track 512.6 -> 509.2 mm
- net ROW5: track 473.0 -> 469.7 mm
- net ROW6: track 505.6 -> 502.3 mm
- net ROW4: track 478.3 -> 475.3 mm
- net ROW3: track 464.2 -> 461.5 mm
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Other:
- board size 430.2 x 139.7 mm -> 430.2 x 141.3 mm

Commit message: RBG Led replaced
Parts:
- J2: value AVR-ISP-6(SWR204-NRTN-D03-RA-GA) -> AVR-ISP-6
- LED1, LED10, LED100, LED101, LED102, LED103, LED104, LED105, LED106, LED107, LED108, LED109, LED11, LED110, LED111, LED12, LED13, LED14, LED15, LED16, LED17, LED18, LED19, LED2, LED20, LED21, LED22, LED23, LED24, LED25, LED26, LED27, LED28, LED29, LED3, LED30, LED31, LED32, LED33, LED34, LED35, LED36, LED37, LED38, LED39, LED4, LED40, LED41, LED42, LED43, LED44, LED45, LED46, LED47, LED48, LED49, LED5, LED50, LED51, LED52, LED53, LED54, LED55, LED56, LED57, LED58, LED59, LED6, LED60, LED61, LED62, LED63, LED64, LED65, LED66, LED67, LED68, LED69, LED7, LED70, LED71, LED72, LED73, LED74, LED75, LED76, LED77, LED78, LED79, LED8, LED80, LED81, LED82, LED83, LED84, LED85, LED86, LED87, LED88, LED89, LED9, LED90, LED91, LED92, LED93, LED94, LED95, LED96, LED97, LED98, LED99: value XZMDKCBDDG45S-9 -> QBLP677R-RGB; footprint SamacSys_Parts:XZMDKCBDDG45S9 -> SamacSys_Parts:QBLP677R-RGB
- moved LED65 371.3 mm to (209.6, 345.3), turned to 0 degrees
- moved LED66 351.9 mm to (228.6, 345.3), turned to 0 degrees
- moved LED67 340.2 mm to (247.7, 345.3)
- moved LED44 333.9 mm to (566.7, 326.2)
- moved LED43 324.3 mm to (566.7, 307.2)
- moved LED80 319.0 mm to (188.1, 364.3)
- moved LED45 317.2 mm to (547.7, 326.2)
- moved LED96 305.0 mm to (178.6, 383.4)
- moved LED42 302.4 mm to (547.6, 307.2)
- moved LED68 302.4 mm to (266.7, 345.3)
- moved LED46 301.6 mm to (528.6, 326.2)
- moved LED82 300.6 mm to (238.1, 364.3)
- moved LED47 297.0 mm to (504.8, 326.2)
- moved LED97 289.9 mm to (202.4, 383.4)
- moved LED81 286.4 mm to (219.1, 364.3)
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Connections:
- LED1 pad 1: SW11 -> SW24
- LED1 pad 2: CS1 -> SW22
- LED1 pad 3: SW12 -> SW23
- LED1 pad 4: SW10 -> CS18
- LED10 pad 1: SW11 -> SW21
- LED10 pad 2: CS10 -> SW19
- LED10 pad 3: SW12 -> SW20
- LED10 pad 4: SW10 -> CS19
- LED100 pad 1: SW14 -> SW3
- LED100 pad 2: CS17 -> SW1
- LED100 pad 3: SW15 -> SW2
- LED100 pad 4: SW13 -> CS5
- LED101 pad 1: SW14 -> SW3
- LED101 pad 2: CS18 -> SW1
- LED101 pad 3: SW15 -> SW2
- LED101 pad 4: SW13 -> CS6
- LED102 pad 1: SW14 -> SW3
- LED102 pad 2: CS19 -> SW1
- LED102 pad 3: SW15 -> SW2
- LED102 pad 4: SW13 -> CS7
- LED103 pad 1: SW14 -> SW3
- LED103 pad 2: CS20 -> SW1
- LED103 pad 3: SW15 -> SW2
- LED103 pad 4: SW13 -> CS8
- LED104 pad 1: SW14 -> SW3
- LED104 pad 2: CS21 -> SW1
- LED104 pad 3: SW15 -> SW2
- LED104 pad 4: SW13 -> CS9
- LED105 pad 1: SW14 -> SW3
- LED105 pad 2: CS22 -> SW1
- LED105 pad 3: SW15 -> SW2
- LED105 pad 4: SW13 -> CS10
- LED106 pad 1: SW14 -> SW3
- LED106 pad 2: CS23 -> SW1
- LED106 pad 3: SW15 -> SW2
- LED106 pad 4: SW13 -> CS11
- LED107 pad 1: SW14 -> SW3
- LED107 pad 2: CS24 -> SW1
- LED107 pad 3: SW15 -> SW2
- LED107 pad 4: SW13 -> CS12
- LED108 pad 1: SW14 -> SW3
- LED108 pad 2: CS25 -> SW1
- LED108 pad 3: SW15 -> SW2
- LED108 pad 4: SW13 -> CS13
- LED109 pad 1: SW14 -> SW3
- LED109 pad 2: CS26 -> SW1
- LED109 pad 3: SW15 -> SW2
- LED109 pad 4: SW13 -> CS14
- LED11 pad 1: SW11 -> SW21
- LED11 pad 2: CS11 -> SW19
- LED11 pad 3: SW12 -> SW20
- LED11 pad 4: SW10 -> CS20
- LED110 pad 1: SW14 -> SW3
- LED110 pad 2: CS27 -> SW1
- LED110 pad 3: SW15 -> SW2
- LED110 pad 4: SW13 -> CS15
- LED111 pad 1: SW14 -> SW3
- LED111 pad 2: CS28 -> SW1
- LED111 pad 3: SW15 -> SW2
- LED111 pad 4: SW13 -> CS16
- LED12 pad 1: SW11 -> SW21
- LED12 pad 2: CS12 -> SW19
- LED12 pad 3: SW12 -> SW20
- LED12 pad 4: SW10 -> CS21
- LED13 pad 1: SW11 -> SW21
- LED13 pad 2: CS13 -> SW19
- LED13 pad 3: SW12 -> SW20
- LED13 pad 4: SW10 -> CS22
- LED14 pad 1: SW11 -> SW21
- LED14 pad 2: CS14 -> SW19
- LED14 pad 3: SW12 -> SW20
- LED14 pad 4: SW10 -> CS23
- LED15 pad 1: SW11 -> SW21
- LED15 pad 2: CS15 -> SW19
- LED15 pad 3: SW12 -> SW20
- LED15 pad 4: SW10 -> CS24
- LED16 pad 1: SW11 -> SW21
- LED16 pad 2: CS16 -> SW19
- LED16 pad 3: SW12 -> SW20
- LED16 pad 4: SW10 -> CS25
- LED17 pad 1: SW8 -> SW21
- LED17 pad 2: CS1 -> SW19
- LED17 pad 3: SW9 -> SW20
- LED17 pad 4: SW7 -> CS26
- LED18 pad 1: SW8 -> SW21
- LED18 pad 2: CS2 -> SW19
- LED18 pad 3: SW9 -> SW20
- LED18 pad 4: SW7 -> CS27
- LED19 pad 1: SW8 -> SW21
- LED19 pad 2: CS3 -> SW19
- LED19 pad 3: SW9 -> SW20
- LED19 pad 4: SW7 -> CS28
- LED2 pad 1: SW11 -> SW24
- LED2 pad 2: CS2 -> SW22
- LED2 pad 3: SW12 -> SW23
- LED2 pad 4: SW10 -> CS19
- LED20 pad 1: SW8 -> SW21
- LED20 pad 2: CS4 -> SW19
- LED20 pad 3: SW9 -> SW20
- LED20 pad 4: SW7 -> CS29
- LED21 pad 1: SW8 -> SW21
- LED21 pad 2: CS5 -> SW19
- LED21 pad 3: SW9 -> SW20
- LED21 pad 4: SW7 -> CS30
- LED22 pad 1: SW8 -> SW21
- LED22 pad 2: CS6 -> SW19
- LED22 pad 3: SW9 -> SW20
- LED22 pad 4: SW7 -> CS31
- LED23 pad 1: SW8 -> SW21
- LED23 pad 2: CS7 -> SW19
- LED23 pad 3: SW9 -> SW20
- LED23 pad 4: SW7 -> CS32
- LED24 pad 1: SW8 -> SW18
- LED24 pad 2: CS8 -> SW16
- LED24 pad 3: SW9 -> SW17
- LED24 pad 4: SW7 -> CS17
- LED25 pad 1: SW8 -> SW18
- LED25 pad 2: CS9 -> SW16
- LED25 pad 3: SW9 -> SW17
- LED25 pad 4: SW7 -> CS18
- LED26 pad 1: SW8 -> SW18
- LED26 pad 2: CS10 -> SW16
- LED26 pad 3: SW9 -> SW17
- LED26 pad 4: SW7 -> CS19
- LED27 pad 1: SW8 -> SW18
- LED27 pad 2: CS11 -> SW16
- LED27 pad 3: SW9 -> SW17
- LED27 pad 4: SW7 -> CS20
- LED28 pad 1: SW8 -> SW18
- LED28 pad 2: CS12 -> SW16
- LED28 pad 3: SW9 -> SW17
- LED28 pad 4: SW7 -> CS21
- LED29 pad 1: SW8 -> SW18
- LED29 pad 2: CS13 -> SW16
- LED29 pad 3: SW9 -> SW17
- LED29 pad 4: SW7 -> CS22
- LED3 pad 1: SW11 -> SW24
- LED3 pad 2: CS3 -> SW22
- LED3 pad 3: SW12 -> SW23
- LED3 pad 4: SW10 -> CS20
- LED30 pad 1: SW8 -> SW18
- LED30 pad 2: CS14 -> SW16
- LED30 pad 3: SW9 -> SW17
- LED30 pad 4: SW7 -> CS23
- LED31 pad 1: SW8 -> SW18
- LED31 pad 2: CS15 -> SW16
- LED31 pad 3: SW9 -> SW17
- LED31 pad 4: SW7 -> CS24
- LED32 pad 1: SW8 -> SW18
- LED32 pad 2: CS16 -> SW16
- LED32 pad 3: SW9 -> SW17
- LED32 pad 4: SW7 -> CS25
- LED33 pad 1: SW5 -> SW18
- LED33 pad 2: CS1 -> SW16
- LED33 pad 3: SW6 -> SW17
- LED33 pad 4: SW4 -> CS26
- LED34 pad 1: SW5 -> SW18
- LED34 pad 2: CS2 -> SW16
- LED34 pad 3: SW6 -> SW17
- LED34 pad 4: SW4 -> CS27
- LED35 pad 1: SW5 -> SW18
- LED35 pad 2: CS3 -> SW16
- LED35 pad 3: SW6 -> SW17
- LED35 pad 4: SW4 -> CS28
- LED36 pad 1: SW5 -> SW18
- LED36 pad 2: CS4 -> SW16
- LED36 pad 3: SW6 -> SW17
- LED36 pad 4: SW4 -> CS29
- LED37 pad 1: SW5 -> SW18
- LED37 pad 2: CS5 -> SW16
- LED37 pad 3: SW6 -> SW17
- LED37 pad 4: SW4 -> CS30
- LED38 pad 1: SW5 -> SW18
- LED38 pad 2: CS6 -> SW16
- LED38 pad 3: SW6 -> SW17
- LED38 pad 4: SW4 -> CS31
- LED39 pad 1: SW5 -> SW18
- LED39 pad 2: CS7 -> SW16
- LED39 pad 3: SW6 -> SW17
- LED39 pad 4: SW4 -> CS32
- LED4 pad 1: SW11 -> SW24
- LED4 pad 2: CS4 -> SW22
- LED4 pad 3: SW12 -> SW23
- LED4 pad 4: SW10 -> CS21
- LED40 pad 1: SW5 -> SW15
- LED40 pad 2: CS8 -> SW13
- LED40 pad 3: SW6 -> SW14
- LED40 pad 4: SW4 -> CS25
- LED41 pad 1: SW5 -> SW15
- LED41 pad 2: CS9 -> SW13
- LED41 pad 3: SW6 -> SW14
- LED41 pad 4: SW4 -> CS26
- LED42 pad 1: SW5 -> SW15
- LED42 pad 2: CS10 -> SW13
- LED42 pad 3: SW6 -> SW14
- LED42 pad 4: SW4 -> CS27
- LED43 pad 1: SW5 -> SW15
- LED43 pad 2: CS11 -> SW13
- LED43 pad 3: SW6 -> SW14
- LED43 pad 4: SW4 -> CS28
- LED44 pad 1: SW5 -> SW15
- LED44 pad 2: CS12 -> SW13
- LED44 pad 3: SW6 -> SW14
- LED44 pad 4: SW4 -> CS29
- LED45 pad 1: SW5 -> SW15
- LED45 pad 2: CS13 -> SW13
- LED45 pad 3: SW6 -> SW14
- LED45 pad 4: SW4 -> CS30
- LED46 pad 1: SW5 -> SW15
- LED46 pad 2: CS14 -> SW13
- LED46 pad 3: SW6 -> SW14
- LED46 pad 4: SW4 -> CS31
- LED47 pad 1: SW5 -> SW15
- LED47 pad 2: CS15 -> SW13
- LED47 pad 3: SW6 -> SW14
- LED47 pad 4: SW4 -> CS32
- LED48 pad 1: SW5 -> SW12
- LED48 pad 2: CS16 -> SW10
- LED48 pad 3: SW6 -> SW11
- LED48 pad 4: SW4 -> CS1
- LED49 pad 1: SW2 -> SW12
- LED49 pad 2: CS1 -> SW10
- LED49 pad 3: SW3 -> SW11
- LED49 pad 4: SW1 -> CS2
- LED5 pad 1: SW11 -> SW24
- LED5 pad 2: CS5 -> SW22
- LED5 pad 3: SW12 -> SW23
- LED5 pad 4: SW10 -> CS30
- LED50 pad 1: SW2 -> SW12
- LED50 pad 2: CS2 -> SW10
- LED50 pad 3: SW3 -> SW11
- LED50 pad 4: SW1 -> CS3
- LED51 pad 1: SW2 -> SW12
- LED51 pad 2: CS3 -> SW10
- LED51 pad 3: SW3 -> SW11
- LED51 pad 4: SW1 -> CS4
- LED52 pad 1: SW2 -> SW12
- LED52 pad 2: CS4 -> SW10
- LED52 pad 3: SW3 -> SW11
- LED52 pad 4: SW1 -> CS5
- LED53 pad 1: SW2 -> SW12
- LED53 pad 2: CS5 -> SW10
- LED53 pad 3: SW3 -> SW11
- LED53 pad 4: SW1 -> CS6
- LED54 pad 1: SW2 -> SW12
- LED54 pad 2: CS6 -> SW10
- LED54 pad 3: SW3 -> SW11
- LED54 pad 4: SW1 -> CS7
- LED55 pad 1: SW2 -> SW12
- LED55 pad 2: CS7 -> SW10
- LED55 pad 3: SW3 -> SW11
- LED55 pad 4: SW1 -> CS8
- LED56 pad 1: SW2 -> SW12
- LED56 pad 2: CS8 -> SW10
- LED56 pad 3: SW3 -> SW11
- LED56 pad 4: SW1 -> CS9
- LED57 pad 1: SW2 -> SW12
- LED57 pad 2: CS9 -> SW10
- LED57 pad 3: SW3 -> SW11
- LED57 pad 4: SW1 -> CS10
- LED58 pad 1: SW2 -> SW12
- LED58 pad 2: CS10 -> SW10
- LED58 pad 3: SW3 -> SW11
- LED58 pad 4: SW1 -> CS11
- LED59 pad 1: SW2 -> SW12
- LED59 pad 2: CS11 -> SW10
- LED59 pad 3: SW3 -> SW11
- LED59 pad 4: SW1 -> CS12
- LED6 pad 1: SW11 -> SW24
- LED6 pad 2: CS6 -> SW22
- LED6 pad 3: SW12 -> SW23
- LED6 pad 4: SW10 -> CS31
- LED60 pad 1: SW2 -> SW12
- LED60 pad 2: CS12 -> SW10
- LED60 pad 3: SW3 -> SW11
- LED60 pad 4: SW1 -> CS13
- LED61 pad 1: SW2 -> SW12
- LED61 pad 2: CS13 -> SW10
- LED61 pad 3: SW3 -> SW11
- LED61 pad 4: SW1 -> CS14
- LED62 pad 1: SW2 -> SW12
- LED62 pad 2: CS14 -> SW10
- LED62 pad 3: SW3 -> SW11
- LED62 pad 4: SW1 -> CS15
- LED63 pad 1: SW2 -> SW12
- LED63 pad 2: CS15 -> SW10
- LED63 pad 3: SW3 -> SW11
- LED63 pad 4: SW1 -> CS16
- LED64 pad 1: SW2 -> SW9
- LED64 pad 2: CS16 -> SW7
- LED64 pad 3: SW3 -> SW8
- LED64 pad 4: SW1 -> CS1
- LED65 pad 1: SW23 -> SW9
- LED65 pad 2: CS17 -> SW7
- LED65 pad 3: SW24 -> SW8
- LED65 pad 4: SW22 -> CS2
- LED66 pad 1: SW23 -> SW9
- LED66 pad 2: CS18 -> SW7
- LED66 pad 3: SW24 -> SW8
- LED66 pad 4: SW22 -> CS3
- LED67 pad 1: SW23 -> SW9
- LED67 pad 2: CS19 -> SW7
- LED67 pad 3: SW24 -> SW8
- LED67 pad 4: SW22 -> CS4
- LED68 pad 1: SW23 -> SW9
- LED68 pad 2: CS20 -> SW7
- LED68 pad 3: SW24 -> SW8
- LED68 pad 4: SW22 -> CS5
- LED69 pad 1: SW23 -> SW9
- LED69 pad 2: CS21 -> SW7
- LED69 pad 3: SW24 -> SW8
- LED69 pad 4: SW22 -> CS6
- LED7 pad 1: SW11 -> SW24
- LED7 pad 2: CS7 -> SW22
- LED7 pad 3: SW12 -> SW23
- LED7 pad 4: SW10 -> CS32
- LED70 pad 1: SW23 -> SW9
- LED70 pad 2: CS22 -> SW7
- LED70 pad 3: SW24 -> SW8
- LED70 pad 4: SW22 -> CS7
- LED71 pad 1: SW23 -> SW9
- LED71 pad 2: CS23 -> SW7
- LED71 pad 3: SW24 -> SW8
- LED71 pad 4: SW22 -> CS8
- LED72 pad 1: SW23 -> SW9
- LED72 pad 2: CS24 -> SW7
- LED72 pad 3: SW24 -> SW8
- LED72 pad 4: SW22 -> CS9
- LED73 pad 1: SW23 -> SW9
- LED73 pad 2: CS25 -> SW7
- LED73 pad 3: SW24 -> SW8
- LED73 pad 4: SW22 -> CS10
- LED74 pad 1: SW23 -> SW9
- LED74 pad 2: CS26 -> SW7
- LED74 pad 3: SW24 -> SW8
- LED74 pad 4: SW22 -> CS11
- LED75 pad 1: SW23 -> SW9
- LED75 pad 2: CS27 -> SW7
- LED75 pad 3: SW24 -> SW8
- LED75 pad 4: SW22 -> CS12
- LED76 pad 1: SW20 -> SW9
- LED76 pad 2: CS17 -> SW7
- LED76 pad 3: SW21 -> SW8
- LED76 pad 4: SW19 -> CS13
- LED77 pad 1: SW20 -> SW9
- LED77 pad 2: CS18 -> SW7
- LED77 pad 3: SW21 -> SW8
- LED77 pad 4: SW19 -> CS14
- LED78 pad 1: SW20 -> SW9
- LED78 pad 2: CS19 -> SW7
- LED78 pad 3: SW21 -> SW8
- LED78 pad 4: SW19 -> CS15
- LED79 pad 1: SW20 -> SW9
- LED79 pad 2: CS20 -> SW7
- LED79 pad 3: SW21 -> SW8
- LED79 pad 4: SW19 -> CS16
- LED8 pad 1: SW11 -> SW21
- LED8 pad 2: CS8 -> SW19
- LED8 pad 3: SW12 -> SW20
- LED8 pad 4: SW10 -> CS17
- LED80 pad 1: SW20 -> SW6
- LED80 pad 2: CS21 -> SW4
- LED80 pad 3: SW21 -> SW5
- LED80 pad 4: SW19 -> CS1
- LED81 pad 1: SW20 -> SW6
- LED81 pad 2: CS22 -> SW4
- LED81 pad 3: SW21 -> SW5
- LED81 pad 4: SW19 -> CS2
- LED82 pad 1: SW20 -> SW6
- LED82 pad 2: CS23 -> SW4
- LED82 pad 3: SW21 -> SW5
- LED82 pad 4: SW19 -> CS3
- LED83 pad 1: SW20 -> SW6
- LED83 pad 2: CS24 -> SW4
- LED83 pad 3: SW21 -> SW5
- LED83 pad 4: SW19 -> CS4
- LED84 pad 1: SW20 -> SW6
- LED84 pad 2: CS25 -> SW4
- LED84 pad 3: SW21 -> SW5
- LED84 pad 4: SW19 -> CS5
- LED85 pad 1: SW20 -> SW6
- LED85 pad 2: CS26 -> SW4
- LED85 pad 3: SW21 -> SW5
- LED85 pad 4: SW19 -> CS6
- LED86 pad 1: SW20 -> SW6
- LED86 pad 2: CS27 -> SW4
- LED86 pad 3: SW21 -> SW5
- LED86 pad 4: SW19 -> CS7
- LED87 pad 1: SW20 -> SW6
- LED87 pad 2: CS28 -> SW4
- LED87 pad 3: SW21 -> SW5
- LED87 pad 4: SW19 -> CS8
- LED88 pad 1: SW17 -> SW6
- LED88 pad 2: CS17 -> SW4
- LED88 pad 3: SW18 -> SW5
- LED88 pad 4: SW16 -> CS9
- LED89 pad 1: SW17 -> SW6
- LED89 pad 2: CS18 -> SW4
- LED89 pad 3: SW18 -> SW5
- LED89 pad 4: SW16 -> CS10
- LED9 pad 1: SW11 -> SW21
- LED9 pad 2: CS9 -> SW19
- LED9 pad 3: SW12 -> SW20
- LED9 pad 4: SW10 -> CS18
- LED90 pad 1: SW17 -> SW6
- LED90 pad 2: CS19 -> SW4
- LED90 pad 3: SW18 -> SW5
- LED90 pad 4: SW16 -> CS11
- LED91 pad 1: SW17 -> SW6
- LED91 pad 2: CS20 -> SW4
- LED91 pad 3: SW18 -> SW5
- LED91 pad 4: SW16 -> CS12
- LED92 pad 1: SW17 -> SW6
- LED92 pad 2: CS21 -> SW4
- LED92 pad 3: SW18 -> SW5
- LED92 pad 4: SW16 -> CS13
- LED93 pad 1: SW17 -> SW6
- LED93 pad 2: CS22 -> SW4
- LED93 pad 3: SW18 -> SW5
- LED93 pad 4: SW16 -> CS14
- LED94 pad 1: SW17 -> SW6
- LED94 pad 2: CS23 -> SW4
- LED94 pad 3: SW18 -> SW5
- LED94 pad 4: SW16 -> CS15
- LED95 pad 1: SW17 -> SW6
- LED95 pad 2: CS24 -> SW4
- LED95 pad 3: SW18 -> SW5
- LED95 pad 4: SW16 -> CS16
- LED96 pad 1: SW17 -> SW3
- LED96 pad 2: CS25 -> SW1
- LED96 pad 3: SW18 -> SW2
- LED96 pad 4: SW16 -> CS1
- LED97 pad 1: SW17 -> SW3
- LED97 pad 2: CS26 -> SW1
- LED97 pad 3: SW18 -> SW2
- LED97 pad 4: SW16 -> CS2
- LED98 pad 1: SW17 -> SW3
- LED98 pad 2: CS27 -> SW1
- LED98 pad 3: SW18 -> SW2
- LED98 pad 4: SW16 -> CS3
- LED99 pad 1: SW17 -> SW3
- LED99 pad 2: CS28 -> SW1
- LED99 pad 3: SW18 -> SW2
- LED99 pad 4: SW16 -> CS4
- SLAVE_U1 pad 30: Net-(SLAVE_U1-Pad30) -> CS29
- SLAVE_U1 pad 31: Net-(SLAVE_U1-Pad31) -> CS30
- SLAVE_U1 pad 32: Net-(SLAVE_U1-Pad32) -> CS31
- SLAVE_U1 pad 33: Net-(SLAVE_U1-Pad33) -> CS32

Commit message: Updated RGB Led footprint and more routing
Parts:
- moved R7 214.9 mm to (593.3, 259.7)
- moved R4 214.9 mm to (579.6, 259.7)
- moved U1 214.9 mm to (586.4, 259.6)
- moved USB1 214.9 mm to (586.4, 247.0)
- moved F1 212.3 mm to (575.1, 257.0)
- moved R10 204.5 mm to (567.6, 287.5)
- moved U3 204.5 mm to (573.5, 287.5)
- moved C24 204.5 mm to (578.4, 287.3)
- moved R11 204.5 mm to (581.4, 286.8)
- moved R12 204.5 mm to (581.4, 288.3)
- moved C25 202.8 mm to (574.5, 265.8)
- moved U4 202.8 mm to (574.2, 271.1)
- moved J2 36.0 mm to (590.0, 287.8), turned to 90 degrees
- moved R2 20.6 mm to (541.1, 259.1), turned to 0 degrees
- moved R3 20.4 mm to (541.2, 261.1), turned to 0 degrees
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Routing:
- net SW3: track 0.00 -> 792.6 mm, vias 0 -> 34
- net SW2: track 0.00 -> 767.5 mm, vias 0 -> 32
- net SW1: track 0.00 -> 733.9 mm, vias 0 -> 32
- net SW6: track 0.00 -> 506.7 mm, vias 0 -> 32
- net SW9: track 0.00 -> 502.2 mm, vias 0 -> 32
- net SW8: track 0.00 -> 493.0 mm, vias 0 -> 32
- net SW5: track 0.00 -> 489.3 mm, vias 0 -> 32
- net SW21: track 0.00 -> 471.2 mm, vias 0 -> 32
- net SW7: track 0.00 -> 450.0 mm, vias 0 -> 32
- net SW4: track 0.00 -> 447.8 mm, vias 0 -> 32
- net SW18: track 0.00 -> 428.2 mm, vias 0 -> 32
- net SW12: track 0.00 -> 422.1 mm, vias 0 -> 32
- net SW17: track 0.00 -> 417.4 mm, vias 0 -> 32
- net SW11: track 0.01 -> 407.0 mm, vias 0 -> 32
- net SW16: track 6.34 -> 376.0 mm, vias 0 -> 32
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
Commit message: Almost done, some routing left
Parts:
- moved R13 2.03 mm to (408.4, 265.2)
- moved R14 1.97 mm to (408.4, 267.1)
- moved R1 1.52 mm to (547.6, 264.7)
- moved R11 0.51 mm to (581.4, 286.3)
- moved C16 0.50 mm to (420.5, 253.2)
- moved C26 0.34 mm to (324.2, 253.7)
- moved C27 0.34 mm to (322.2, 253.7)
- moved C15 0.28 mm to (548.3, 274.1)
Routing:
- net +5V: track 0.00 -> 460.7 mm, vias 0 -> 8
- net GND: track 2.98 -> 368.7 mm, vias 0 -> 32
- net CS28: track 62.5 -> 367.9 mm, vias 4 -> 14
- net SDA_3.3: track 0.00 -> 304.8 mm, vias 0 -> 7
- net CS25: track 50.9 -> 355.0 mm, vias 6 -> 18
- net SCL_3.3: track 0.00 -> 302.5 mm, vias 0 -> 6
- net CS26: track 60.0 -> 361.4 mm, vias 6 -> 15
- net CS27: track 59.8 -> 359.1 mm, vias 6 -> 15
- net SW4: track 447.8 -> 726.8 mm, vias 32 -> 36
- net SW5: track 489.3 -> 766.6 mm, vias 32 -> 36
- net CS17: track 27.7 -> 290.9 mm, vias 2 -> 5
- net CS16: track 188.5 -> 440.6 mm, vias 7 -> 10
- net CS29: track 58.4 -> 303.8 mm, vias 4 -> 11
- net CS19: track 61.9 -> 295.1 mm, vias 5 -> 10
- net SW10: track 365.9 -> 592.4 mm, vias 32 -> 33
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