File: TooManyKeys/Matrix.sch (KiCad schematic (older format))
At the start: 222 parts

Commit message: Final Schematic version, starting work on pcb
Parts:
- MX_0, MX_1, MX_2, MX_3, MX_4, MX_5, MX_6, MX_7, MX_8, MX_9, MX_A1, MX_B1, MX_BSLS1, MX_BSPC1, MX_C1, MX_CAPS1, MX_COMM1, MX_D1, MX_DEL1, MX_DOT1, MX_DOWN1, MX_E1, MX_END1, MX_ENT1, MX_EQL1, MX_ESC1, MX_F1, MX_F10, MX_F11, MX_F12, MX_F13, MX_F2, MX_F3, MX_F4, MX_F5, MX_F6, MX_F7, MX_F8, MX_F9, MX_G1, MX_GRV1, MX_H1, MX_HOME1, MX_I1, MX_INS1, MX_J1, MX_K1, MX_L1, MX_LALT1, MX_LBRC1, MX_LCTL1, MX_LEFT1, MX_LGUI1, MX_LSFT1, MX_M1, MX_MENU1, MX_MINS1, MX_MUTE1, MX_N1, MX_NEXT1, MX_NLCK1, MX_O1, MX_P*1, MX_P+1, MX_P-1, MX_P/1, MX_P0, MX_P1, MX_P10, MX_P2, MX_P3, MX_P4, MX_P5, MX_P6, MX_P7, MX_P8, MX_P9, MX_PAUSE1, MX_PDOT1, MX_PENT1, MX_PGDN1, MX_PGUP1, MX_PLAY1, MX_PREV1, MX_PSCR1, MX_Q1, MX_QUOT1, MX_R1, MX_RALT1, MX_RBRC1, MX_RCTL1, MX_RGHT1, MX_RGUI1, MX_RSFT1, MX_S1, MX_SCLN1, MX_SLCK1, MX_SLSH1, MX_SPC1, MX_STOP1, MX_T1, MX_TAB1, MX_U1, MX_UP1, MX_V1, MX_VOLD1, MX_VOLU1, MX_W1, MX_X1, MX_Y1, MX_Z1: symbol MX_Alps_Hybrid:MX-NoLED -> TooManyKeys-rescue:MX-NoLED-MX_Alps_Hybrid
Connections:
- net ROW0: now also D1.1 (K), D2.1 (K), D3.1 (K), D4.1 (K), D5.1 (K), D6.1 (K), D7.1 (K)

Commit message: New footprint, pcb key matrix completed
Changed lines of the file:
@@
 $Descr B 17000 11000
 encoding utf-8
-Sheet 2 3
+Sheet 3 3
 Title ""
 Date ""
@@
 Connection ~ 12500 3550
 Connection ~ 13050 3550
-Text GLabel 800  2900 0    50   Input ~ 0
-ROW2
 Connection ~ 9200 4200
 Wire Wire Line
@@
 Text GLabel 800  3550 0    50   Input ~ 0
 ROW3
-Text GLabel 11750 1000 1    50   Input ~ 0
-COL18
 Connection ~ 8100 2250
 Wire Wire Line
