File: TooManyKeys/Led.sch (KiCad schematic (older format))
At the start: 2 parts

Commit message: adding IS31FL3733-TQ to led sch
Parts:
- removed LED?: WS2812B, symbol ws2812b:WS2812B
- removed R?: 500, symbol Device:R_Small
- added U? (x2): IS31FL3733-TQ, Package_QFP:TQFP-48-1EP_7x7mm_P0.5mm_EP5x5mm, symbol Driver_LED:IS31FL3733-TQ
Connections:
- net labels added: +5V, GND, SCL, SDA
- net labels removed: LED
- wire segments 2 -> 3
Changed lines of the file:
@@
 $EndDescr
 $Comp
-L Device:R_Small R?
-U 1 1 60658413
-P 1600 1100
-F 0 "R?" V 1404 1100 50  0000 C CNN
-F 1 "500" V 1495 1100 50  0000 C CNN
-F 2 "" H 1600 1100 50  0001 C CNN
-F 3 "~" H 1600 1100 50  0001 C CNN
-	1    1600 1100
-	0    1    1    0
+L Driver_LED:IS31FL3733-TQ U?
+U 1 1 5E8737CD
+P 2300 2950
+F 0 "U?" H 2300 1261 50  0000 C CNN
+F 1 "IS31FL3733-TQ" H 2300 1170 50  0000 C CNN
+F 2 "Package_QFP:TQFP-48-1EP_7x7mm_P0.5mm_EP5x5mm" H 2300 2950 50  0001 C CNN
+F 3 "http://www.issi.com/WW/pdf/IS31FL3733.pdf" H 2300 2950 50  0001 C CNN
+	1    2300 2950
+	1    0    0    -1
 $EndComp
-Text GLabel 1300 1100 0    50   Input ~ 0
-LED
-Wire Wire Line
-	1300 1100 1500 1100
 $Comp
-L ws2812b:WS2812B LED?
-U 1 1 606596C0
-P 2450 1300
-F 0 "LED?" H 2450 1787 60  0000 C CNN
-F 1 "WS2812B" H 2450 1681 60  0000 C CNN
-F 2 "" V 2400 1300 60  0000 C CNN
-F 3 "" V 2400 1300 60  0000 C CNN
-	1    2450 1300
-	-1   0    0    -1
+L Driver_LED:IS31FL3733-TQ U?
+U 1 1 5E87B1A0
+P 4650 5850
+F 0 "U?" H 4650 4161 50  0000 C CNN
+F 1 "IS31FL3733-TQ" H 4650 4070 50  0000 C CNN
+F 2 "Package_QFP:TQFP-48-1EP_7x7mm_P0.5mm_EP5x5mm" H 4650 5850 50  0001 C CNN
+F 3 "http://www.issi.com/WW/pdf/IS31FL3733.pdf" H 4650 5850 50  0001 C CNN
+	1    4650 5850
+	1    0    0    -1
+$EndComp
+$Comp
+L power:GND #PWR?
+U 1 1 5E87F64E
+P 1250 2650
+F 0 "#PWR?" H 1250 2400 50  0001 C CNN
+F 1 "GND" H 1255 2477 50  0000 C CNN
+F 2 "" H 1250 2650 50  0001 C CNN
+F 3 "" H 1250 2650 50  0001 C CNN
+	1    1250 2650
+	1    0    0    -1
 $EndComp
 Wire Wire Line
-	1700 1100 1950 1100
+	1600 2550 1250 2550
+Wire Wire Line
+	1250 2550 1250 2650
+Wire Wire Line
+	1600 2650 1250 2650
+Connection ~ 1250 2650
+Text GLabel 1600 1750 0    50   Input ~ 0
+SDA
+Text GLabel 1600 1850 0    50   Input ~ 0
+SCL
+$Comp
+L power:+5V #PWR?
+U 1 1 5E882C24
+P 1250 1400
+F 0 "#PWR?" H 1250 1250 50  0001 C CNN
+F 1 "+5V" H 1265 1573 50  0000 C CNN
+F 2 "" H 1250 1400 50  0001 C CNN
+F 3 "" H 1250 1400 50  0001 C CNN
+	1    1250 1400
+	1    0    0    -1
+$EndComp
 $EndSCHEMATC

Commit message: led work
Parts:
- removed U?: IS31FL3733-TQ, Package_QFP:TQFP-48-1EP_7x7mm_P0.5mm_EP5x5mm, symbol Driver_LED:IS31FL3733-TQ
- added C? (x8): 0.47uF, symbol Device:C_Small
- added C? (x6): 0.1uF, symbol Device:C_Small
- added R? (x2): 100k, symbol Device:R_Small
- added R? (x2): 20k, symbol Device:R_Small
- added R? (x2): 10k, symbol Device:R_Small
- added U?: IS31FL3733-TQ, Package_QFP:TQFP-48-1EP_7x7mm_P0.5mm_EP5x5mm, symbol Driver_LED:IS31FL3733-TQ
Connections:
- net +5V: now also U?.20 (PVCC), U?.29 (PVCC), U?.37 (AVCC), U?.38 (DVCC), U?.39 (VIO), C?.1, C?.1, C?.1, C?.1, C?.1, C?.1, C?.1, C?.1, C?.1, C?.1, C?.1, C?.1, C?.1, C?.1, R?.2, R?.2, U?.20 (PVCC), U?.29 (PVCC), U?.37 (AVCC), U?.38 (DVCC), U?.39 (VIO), U?.43 (ADDR1)
- net GND: now also U?.12 (PGND), U?.34 (AGND), U?.48 (GND), U?.49 (GND), U?.5 (PGND), C?.2, C?.2, C?.2, C?.2, C?.2, C?.2, C?.2, C?.2, C?.2, C?.2, C?.2, C?.2, C?.2, C?.2, R?.2, R?.2, R?.2, R?.2, U?.12 (PGND), U?.34 (AGND), U?.44 (ADDR2), U?.48 (GND), U?.49 (GND), U?.5 (PGND)
- net SCL: now also U?.42 (SCL)
- net SDA: now also U?.41 (SDA)
- net at U?.35 (RSET): now also R?.1
- net at U?.46 (~SDB): now also R?.1
- net at U?.47 (IICRST): now also R?.1
- new net: R?.1, U?.35 (RSET)
- new net: R?.1, U?.46 (~SDB)
- new net: R?.1, U?.47 (IICRST)
Other:
- moved on the sheet: U?

Commit message: Adding led matrix
Parts:
- added LED? (x64): XZMDKCBDDG45S-9, XZMDKCBDDG45S9, symbol SamacSys_Parts:XZMDKCBDDG45S-9
Connections:
- new net CS1: LED?.2 (COMMON_ANODE), LED?.2 (COMMON_ANODE), LED?.2 (COMMON_ANODE), LED?.2 (COMMON_ANODE)
- new net CS10: LED?.2 (COMMON_ANODE), LED?.2 (COMMON_ANODE), LED?.2 (COMMON_ANODE), LED?.2 (COMMON_ANODE)
- new net CS11: LED?.2 (COMMON_ANODE), LED?.2 (COMMON_ANODE), LED?.2 (COMMON_ANODE), LED?.2 (COMMON_ANODE)
- new net CS12: LED?.2 (COMMON_ANODE), LED?.2 (COMMON_ANODE), LED?.2 (COMMON_ANODE), LED?.2 (COMMON_ANODE)
- new net CS13: LED?.2 (COMMON_ANODE), LED?.2 (COMMON_ANODE), LED?.2 (COMMON_ANODE), LED?.2 (COMMON_ANODE)
- new net CS14: LED?.2 (COMMON_ANODE), LED?.2 (COMMON_ANODE), LED?.2 (COMMON_ANODE), LED?.2 (COMMON_ANODE)
- new net CS15: LED?.2 (COMMON_ANODE), LED?.2 (COMMON_ANODE), LED?.2 (COMMON_ANODE), LED?.2 (COMMON_ANODE)
- new net CS16: LED?.2 (COMMON_ANODE), LED?.2 (COMMON_ANODE), LED?.2 (COMMON_ANODE), LED?.2 (COMMON_ANODE)
- new net CS2: LED?.2 (COMMON_ANODE), LED?.2 (COMMON_ANODE), LED?.2 (COMMON_ANODE), LED?.2 (COMMON_ANODE)
- new net CS3: LED?.2 (COMMON_ANODE), LED?.2 (COMMON_ANODE), LED?.2 (COMMON_ANODE), LED?.2 (COMMON_ANODE)
- new net CS4: LED?.2 (COMMON_ANODE), LED?.2 (COMMON_ANODE), LED?.2 (COMMON_ANODE), LED?.2 (COMMON_ANODE)
- new net CS5: LED?.2 (COMMON_ANODE), LED?.2 (COMMON_ANODE), LED?.2 (COMMON_ANODE), LED?.2 (COMMON_ANODE)
- new net CS6: LED?.2 (COMMON_ANODE), LED?.2 (COMMON_ANODE), LED?.2 (COMMON_ANODE), LED?.2 (COMMON_ANODE)
- new net CS7: LED?.2 (COMMON_ANODE), LED?.2 (COMMON_ANODE), LED?.2 (COMMON_ANODE), LED?.2 (COMMON_ANODE)
- new net CS8: LED?.2 (COMMON_ANODE), LED?.2 (COMMON_ANODE), LED?.2 (COMMON_ANODE), LED?.2 (COMMON_ANODE)
- new net CS9: LED?.2 (COMMON_ANODE), LED?.2 (COMMON_ANODE), LED?.2 (COMMON_ANODE), LED?.2 (COMMON_ANODE)
- new net SW1: LED?.4 (CATHODE_GREEN), LED?.4 (CATHODE_GREEN), LED?.4 (CATHODE_GREEN), LED?.4 (CATHODE_GREEN), LED?.4 (CATHODE_GREEN), LED?.4 (CATHODE_GREEN), LED?.4 (CATHODE_GREEN), LED?.4 (CATHODE_GREEN), LED?.4 (CATHODE_GREEN), LED?.4 (CATHODE_GREEN), LED?.4 (CATHODE_GREEN), LED?.4 (CATHODE_GREEN), LED?.4 (CATHODE_GREEN), LED?.4 (CATHODE_GREEN), LED?.4 (CATHODE_GREEN), LED?.4 (CATHODE_GREEN)
- new net SW10: LED?.4 (CATHODE_GREEN), LED?.4 (CATHODE_GREEN), LED?.4 (CATHODE_GREEN), LED?.4 (CATHODE_GREEN), LED?.4 (CATHODE_GREEN), LED?.4 (CATHODE_GREEN), LED?.4 (CATHODE_GREEN), LED?.4 (CATHODE_GREEN), LED?.4 (CATHODE_GREEN), LED?.4 (CATHODE_GREEN), LED?.4 (CATHODE_GREEN), LED?.4 (CATHODE_GREEN), LED?.4 (CATHODE_GREEN), LED?.4 (CATHODE_GREEN), LED?.4 (CATHODE_GREEN), LED?.4 (CATHODE_GREEN)
- new net SW11: LED?.1 (CATHODE_RED), LED?.1 (CATHODE_RED), LED?.1 (CATHODE_RED), LED?.1 (CATHODE_RED), LED?.1 (CATHODE_RED), LED?.1 (CATHODE_RED), LED?.1 (CATHODE_RED), LED?.1 (CATHODE_RED), LED?.1 (CATHODE_RED), LED?.1 (CATHODE_RED), LED?.1 (CATHODE_RED), LED?.1 (CATHODE_RED), LED?.1 (CATHODE_RED), LED?.1 (CATHODE_RED), LED?.1 (CATHODE_RED), LED?.1 (CATHODE_RED)
- new net SW12: LED?.3 (CATHODE_BLUE), LED?.3 (CATHODE_BLUE), LED?.3 (CATHODE_BLUE), LED?.3 (CATHODE_BLUE), LED?.3 (CATHODE_BLUE), LED?.3 (CATHODE_BLUE), LED?.3 (CATHODE_BLUE), LED?.3 (CATHODE_BLUE), LED?.3 (CATHODE_BLUE), LED?.3 (CATHODE_BLUE), LED?.3 (CATHODE_BLUE), LED?.3 (CATHODE_BLUE), LED?.3 (CATHODE_BLUE), LED?.3 (CATHODE_BLUE), LED?.3 (CATHODE_BLUE), LED?.3 (CATHODE_BLUE)
- new net SW2: LED?.1 (CATHODE_RED), LED?.1 (CATHODE_RED), LED?.1 (CATHODE_RED), LED?.1 (CATHODE_RED), LED?.1 (CATHODE_RED), LED?.1 (CATHODE_RED), LED?.1 (CATHODE_RED), LED?.1 (CATHODE_RED), LED?.1 (CATHODE_RED), LED?.1 (CATHODE_RED), LED?.1 (CATHODE_RED), LED?.1 (CATHODE_RED), LED?.1 (CATHODE_RED), LED?.1 (CATHODE_RED), LED?.1 (CATHODE_RED), LED?.1 (CATHODE_RED)
- new net SW3: LED?.3 (CATHODE_BLUE), LED?.3 (CATHODE_BLUE), LED?.3 (CATHODE_BLUE), LED?.3 (CATHODE_BLUE), LED?.3 (CATHODE_BLUE), LED?.3 (CATHODE_BLUE), LED?.3 (CATHODE_BLUE), LED?.3 (CATHODE_BLUE), LED?.3 (CATHODE_BLUE), LED?.3 (CATHODE_BLUE), LED?.3 (CATHODE_BLUE), LED?.3 (CATHODE_BLUE), LED?.3 (CATHODE_BLUE), LED?.3 (CATHODE_BLUE), LED?.3 (CATHODE_BLUE), LED?.3 (CATHODE_BLUE)
- new net SW4: LED?.4 (CATHODE_GREEN), LED?.4 (CATHODE_GREEN), LED?.4 (CATHODE_GREEN), LED?.4 (CATHODE_GREEN), LED?.4 (CATHODE_GREEN), LED?.4 (CATHODE_GREEN), LED?.4 (CATHODE_GREEN), LED?.4 (CATHODE_GREEN), LED?.4 (CATHODE_GREEN), LED?.4 (CATHODE_GREEN), LED?.4 (CATHODE_GREEN), LED?.4 (CATHODE_GREEN), LED?.4 (CATHODE_GREEN), LED?.4 (CATHODE_GREEN), LED?.4 (CATHODE_GREEN), LED?.4 (CATHODE_GREEN)
- new net SW5: LED?.1 (CATHODE_RED), LED?.1 (CATHODE_RED), LED?.1 (CATHODE_RED), LED?.1 (CATHODE_RED), LED?.1 (CATHODE_RED), LED?.1 (CATHODE_RED), LED?.1 (CATHODE_RED), LED?.1 (CATHODE_RED), LED?.1 (CATHODE_RED), LED?.1 (CATHODE_RED), LED?.1 (CATHODE_RED), LED?.1 (CATHODE_RED), LED?.1 (CATHODE_RED), LED?.1 (CATHODE_RED), LED?.1 (CATHODE_RED), LED?.1 (CATHODE_RED)
- new net SW6: LED?.3 (CATHODE_BLUE), LED?.3 (CATHODE_BLUE), LED?.3 (CATHODE_BLUE), LED?.3 (CATHODE_BLUE), LED?.3 (CATHODE_BLUE), LED?.3 (CATHODE_BLUE), LED?.3 (CATHODE_BLUE), LED?.3 (CATHODE_BLUE), LED?.3 (CATHODE_BLUE), LED?.3 (CATHODE_BLUE), LED?.3 (CATHODE_BLUE), LED?.3 (CATHODE_BLUE), LED?.3 (CATHODE_BLUE), LED?.3 (CATHODE_BLUE), LED?.3 (CATHODE_BLUE), LED?.3 (CATHODE_BLUE)
- new net SW7: LED?.4 (CATHODE_GREEN), LED?.4 (CATHODE_GREEN), LED?.4 (CATHODE_GREEN), LED?.4 (CATHODE_GREEN), LED?.4 (CATHODE_GREEN), LED?.4 (CATHODE_GREEN), LED?.4 (CATHODE_GREEN), LED?.4 (CATHODE_GREEN), LED?.4 (CATHODE_GREEN), LED?.4 (CATHODE_GREEN), LED?.4 (CATHODE_GREEN), LED?.4 (CATHODE_GREEN), LED?.4 (CATHODE_GREEN), LED?.4 (CATHODE_GREEN), LED?.4 (CATHODE_GREEN), LED?.4 (CATHODE_GREEN)
- new net SW8: LED?.1 (CATHODE_RED), LED?.1 (CATHODE_RED), LED?.1 (CATHODE_RED), LED?.1 (CATHODE_RED), LED?.1 (CATHODE_RED), LED?.1 (CATHODE_RED), LED?.1 (CATHODE_RED), LED?.1 (CATHODE_RED), LED?.1 (CATHODE_RED), LED?.1 (CATHODE_RED), LED?.1 (CATHODE_RED), LED?.1 (CATHODE_RED), LED?.1 (CATHODE_RED), LED?.1 (CATHODE_RED), LED?.1 (CATHODE_RED), LED?.1 (CATHODE_RED)
- new net SW9: LED?.3 (CATHODE_BLUE), LED?.3 (CATHODE_BLUE), LED?.3 (CATHODE_BLUE), LED?.3 (CATHODE_BLUE), LED?.3 (CATHODE_BLUE), LED?.3 (CATHODE_BLUE), LED?.3 (CATHODE_BLUE), LED?.3 (CATHODE_BLUE), LED?.3 (CATHODE_BLUE), LED?.3 (CATHODE_BLUE), LED?.3 (CATHODE_BLUE), LED?.3 (CATHODE_BLUE), LED?.3 (CATHODE_BLUE), LED?.3 (CATHODE_BLUE), LED?.3 (CATHODE_BLUE), LED?.3 (CATHODE_BLUE)
Other:
- moved on the sheet: C?, R?, U?

Commit message: V1 Schematics
Parts:
- removed C? (x8): 0.47uF, symbol Device:C_Small
- removed C? (x6): 0.1uF, symbol Device:C_Small
- removed R? (x2): 100k, symbol Device:R_Small
- removed R? (x2): 20k, symbol Device:R_Small
- removed R? (x2): 10k, symbol Device:R_Small
- removed U? (x2): IS31FL3733-TQ, Package_QFP:TQFP-48-1EP_7x7mm_P0.5mm_EP5x5mm, symbol Driver_LED:IS31FL3733-TQ
- added LED? (x47): XZMDKCBDDG45S-9, XZMDKCBDDG45S9, symbol SamacSys_Parts:XZMDKCBDDG45S-9
Connections:
- new net CS17: LED?.2 (COMMON_ANODE), LED?.2 (COMMON_ANODE), LED?.2 (COMMON_ANODE), LED?.2 (COMMON_ANODE)
- new net CS18: LED?.2 (COMMON_ANODE), LED?.2 (COMMON_ANODE), LED?.2 (COMMON_ANODE), LED?.2 (COMMON_ANODE)
- new net CS19: LED?.2 (COMMON_ANODE), LED?.2 (COMMON_ANODE), LED?.2 (COMMON_ANODE), LED?.2 (COMMON_ANODE)
- new net CS20: LED?.2 (COMMON_ANODE), LED?.2 (COMMON_ANODE), LED?.2 (COMMON_ANODE), LED?.2 (COMMON_ANODE)
- new net CS21: LED?.2 (COMMON_ANODE), LED?.2 (COMMON_ANODE), LED?.2 (COMMON_ANODE), LED?.2 (COMMON_ANODE)
- new net CS22: LED?.2 (COMMON_ANODE), LED?.2 (COMMON_ANODE), LED?.2 (COMMON_ANODE), LED?.2 (COMMON_ANODE)
- new net CS23: LED?.2 (COMMON_ANODE), LED?.2 (COMMON_ANODE), LED?.2 (COMMON_ANODE), LED?.2 (COMMON_ANODE)
- new net CS24: LED?.2 (COMMON_ANODE), LED?.2 (COMMON_ANODE), LED?.2 (COMMON_ANODE), LED?.2 (COMMON_ANODE)
- new net CS25: LED?.2 (COMMON_ANODE), LED?.2 (COMMON_ANODE), LED?.2 (COMMON_ANODE), LED?.2 (COMMON_ANODE)
- new net CS26: LED?.2 (COMMON_ANODE), LED?.2 (COMMON_ANODE), LED?.2 (COMMON_ANODE), LED?.2 (COMMON_ANODE)
- new net CS27: LED?.2 (COMMON_ANODE), LED?.2 (COMMON_ANODE), LED?.2 (COMMON_ANODE), LED?.2 (COMMON_ANODE)
- new net CS28: LED?.2 (COMMON_ANODE), LED?.2 (COMMON_ANODE), LED?.2 (COMMON_ANODE)
- new net SW13: LED?.4 (CATHODE_GREEN), LED?.4 (CATHODE_GREEN), LED?.4 (CATHODE_GREEN), LED?.4 (CATHODE_GREEN), LED?.4 (CATHODE_GREEN), LED?.4 (CATHODE_GREEN), LED?.4 (CATHODE_GREEN), LED?.4 (CATHODE_GREEN), LED?.4 (CATHODE_GREEN), LED?.4 (CATHODE_GREEN), LED?.4 (CATHODE_GREEN), LED?.4 (CATHODE_GREEN)
- new net SW14: LED?.1 (CATHODE_RED), LED?.1 (CATHODE_RED), LED?.1 (CATHODE_RED), LED?.1 (CATHODE_RED), LED?.1 (CATHODE_RED), LED?.1 (CATHODE_RED), LED?.1 (CATHODE_RED), LED?.1 (CATHODE_RED), LED?.1 (CATHODE_RED), LED?.1 (CATHODE_RED), LED?.1 (CATHODE_RED), LED?.1 (CATHODE_RED)
- new net SW15: LED?.3 (CATHODE_BLUE), LED?.3 (CATHODE_BLUE), LED?.3 (CATHODE_BLUE), LED?.3 (CATHODE_BLUE), LED?.3 (CATHODE_BLUE), LED?.3 (CATHODE_BLUE), LED?.3 (CATHODE_BLUE), LED?.3 (CATHODE_BLUE), LED?.3 (CATHODE_BLUE), LED?.3 (CATHODE_BLUE), LED?.3 (CATHODE_BLUE), LED?.3 (CATHODE_BLUE)
- new net SW16: LED?.4 (CATHODE_GREEN), LED?.4 (CATHODE_GREEN), LED?.4 (CATHODE_GREEN), LED?.4 (CATHODE_GREEN), LED?.4 (CATHODE_GREEN), LED?.4 (CATHODE_GREEN), LED?.4 (CATHODE_GREEN), LED?.4 (CATHODE_GREEN), LED?.4 (CATHODE_GREEN), LED?.4 (CATHODE_GREEN), LED?.4 (CATHODE_GREEN), LED?.4 (CATHODE_GREEN)
- new net SW17: LED?.1 (CATHODE_RED), LED?.1 (CATHODE_RED), LED?.1 (CATHODE_RED), LED?.1 (CATHODE_RED), LED?.1 (CATHODE_RED), LED?.1 (CATHODE_RED), LED?.1 (CATHODE_RED), LED?.1 (CATHODE_RED), LED?.1 (CATHODE_RED), LED?.1 (CATHODE_RED), LED?.1 (CATHODE_RED), LED?.1 (CATHODE_RED)
- new net SW18: LED?.3 (CATHODE_BLUE), LED?.3 (CATHODE_BLUE), LED?.3 (CATHODE_BLUE), LED?.3 (CATHODE_BLUE), LED?.3 (CATHODE_BLUE), LED?.3 (CATHODE_BLUE), LED?.3 (CATHODE_BLUE), LED?.3 (CATHODE_BLUE), LED?.3 (CATHODE_BLUE), LED?.3 (CATHODE_BLUE), LED?.3 (CATHODE_BLUE), LED?.3 (CATHODE_BLUE)
- new net SW19: LED?.4 (CATHODE_GREEN), LED?.4 (CATHODE_GREEN), LED?.4 (CATHODE_GREEN), LED?.4 (CATHODE_GREEN), LED?.4 (CATHODE_GREEN), LED?.4 (CATHODE_GREEN), LED?.4 (CATHODE_GREEN), LED?.4 (CATHODE_GREEN), LED?.4 (CATHODE_GREEN), LED?.4 (CATHODE_GREEN), LED?.4 (CATHODE_GREEN), LED?.4 (CATHODE_GREEN)
- new net SW20: LED?.1 (CATHODE_RED), LED?.1 (CATHODE_RED), LED?.1 (CATHODE_RED), LED?.1 (CATHODE_RED), LED?.1 (CATHODE_RED), LED?.1 (CATHODE_RED), LED?.1 (CATHODE_RED), LED?.1 (CATHODE_RED), LED?.1 (CATHODE_RED), LED?.1 (CATHODE_RED), LED?.1 (CATHODE_RED), LED?.1 (CATHODE_RED)
- new net SW21: LED?.3 (CATHODE_BLUE), LED?.3 (CATHODE_BLUE), LED?.3 (CATHODE_BLUE), LED?.3 (CATHODE_BLUE), LED?.3 (CATHODE_BLUE), LED?.3 (CATHODE_BLUE), LED?.3 (CATHODE_BLUE), LED?.3 (CATHODE_BLUE), LED?.3 (CATHODE_BLUE), LED?.3 (CATHODE_BLUE), LED?.3 (CATHODE_BLUE), LED?.3 (CATHODE_BLUE)
- new net SW22: LED?.4 (CATHODE_GREEN), LED?.4 (CATHODE_GREEN), LED?.4 (CATHODE_GREEN), LED?.4 (CATHODE_GREEN), LED?.4 (CATHODE_GREEN), LED?.4 (CATHODE_GREEN), LED?.4 (CATHODE_GREEN), LED?.4 (CATHODE_GREEN), LED?.4 (CATHODE_GREEN), LED?.4 (CATHODE_GREEN), LED?.4 (CATHODE_GREEN)
- new net SW23: LED?.1 (CATHODE_RED), LED?.1 (CATHODE_RED), LED?.1 (CATHODE_RED), LED?.1 (CATHODE_RED), LED?.1 (CATHODE_RED), LED?.1 (CATHODE_RED), LED?.1 (CATHODE_RED), LED?.1 (CATHODE_RED), LED?.1 (CATHODE_RED), LED?.1 (CATHODE_RED), LED?.1 (CATHODE_RED)
- new net SW24: LED?.3 (CATHODE_BLUE), LED?.3 (CATHODE_BLUE), LED?.3 (CATHODE_BLUE), LED?.3 (CATHODE_BLUE), LED?.3 (CATHODE_BLUE), LED?.3 (CATHODE_BLUE), LED?.3 (CATHODE_BLUE), LED?.3 (CATHODE_BLUE), LED?.3 (CATHODE_BLUE), LED?.3 (CATHODE_BLUE), LED?.3 (CATHODE_BLUE)

Commit message: WIP pcb
Parts:
- LED1, LED10, LED100, LED101, LED102, LED103, LED104, LED105, LED106, LED107, LED108, LED109, LED11, LED110, LED111, LED12, LED13, LED14, LED15, LED16, LED17, LED18, LED19, LED2, LED20, LED21, LED22, LED23, LED24, LED25, LED26, LED27, LED28, LED29, LED3, LED30, LED31, LED32, LED33, LED34, LED35, LED36, LED37, LED38, LED39, LED4, LED40, LED41, LED42, LED43, LED44, LED45, LED46, LED47, LED48, LED49, LED5, LED50, LED51, LED52, LED53, LED54, LED55, LED56, LED57, LED58, LED59, LED6, LED60, LED61, LED62, LED63, LED64, LED65, LED66, LED67, LED68, LED69, LED7, LED70, LED71, LED72, LED73, LED74, LED75, LED76, LED77, LED78, LED79, LED8, LED80, LED81, LED82, LED83, LED84, LED85, LED86, LED87, LED88, LED89, LED9, LED90, LED91, LED92, LED93, LED94, LED95, LED96, LED97, LED98, LED99: renamed from LED?; footprint XZMDKCBDDG45S9 -> SamacSys_Parts:XZMDKCBDDG45S9

Commit message: Final Schematic version, starting work on pcb
Parts:
- LED1, LED10, LED100, LED101, LED102, LED103, LED104, LED105, LED106, LED107, LED108, LED109, LED11, LED110, LED111, LED12, LED13, LED14, LED15, LED16, LED17, LED18, LED19, LED2, LED20, LED21, LED22, LED23, LED24, LED25, LED26, LED27, LED28, LED29, LED3, LED30, LED31, LED32, LED33, LED34, LED35, LED36, LED37, LED38, LED39, LED4, LED40, LED41, LED42, LED43, LED44, LED45, LED46, LED47, LED48, LED49, LED5, LED50, LED51, LED52, LED53, LED54, LED55, LED56, LED57, LED58, LED59, LED6, LED60, LED61, LED62, LED63, LED64, LED65, LED66, LED67, LED68, LED69, LED7, LED70, LED71, LED72, LED73, LED74, LED75, LED76, LED77, LED78, LED79, LED8, LED80, LED81, LED82, LED83, LED84, LED85, LED86, LED87, LED88, LED89, LED9, LED90, LED91, LED92, LED93, LED94, LED95, LED96, LED97, LED98, LED99: symbol SamacSys_Parts:XZMDKCBDDG45S-9 -> TooManyKeys-rescue:XZMDKCBDDG45S-9-SamacSys_Parts

Commit message: RBG Led replaced
Parts:
- removed LED1, LED10, LED100, LED101, LED102, LED103, LED104, LED105, LED106, LED107, LED108, LED109, LED11, LED110, LED111, LED12, LED13, LED14, LED15, LED16, LED17, LED18, LED19, LED2, LED20, LED21, LED22, LED23, LED24, LED25, LED26, LED27, LED28, LED29, LED3, LED30, LED31, LED32, LED33, LED34, LED35, LED36, LED37, LED38, LED39, LED4, LED40, LED41, LED42, LED43, LED44, LED45, LED46, LED47, LED48, LED49, LED5, LED50, LED51, LED52, LED53, LED54, LED55, LED56, LED57, LED58, LED59, LED6, LED60, LED61, LED62, LED63, LED64, LED65, LED66, LED67, LED68, LED69, LED7, LED70, LED71, LED72, LED73, LED74, LED75, LED76, LED77, LED78, LED79, LED8, LED80, LED81, LED82, LED83, LED84, LED85, LED86, LED87, LED88, LED89, LED9, LED90, LED91, LED92, LED93, LED94, LED95, LED96, LED97, LED98, LED99: XZMDKCBDDG45S-9, SamacSys_Parts:XZMDKCBDDG45S9, symbol TooManyKeys-rescue:XZMDKCBDDG45S-9-SamacSys_Parts
- added LED1, LED10, LED100, LED101, LED102, LED103, LED104, LED105, LED106, LED107, LED108, LED109, LED11, LED110, LED111, LED12, LED13, LED14, LED15, LED16, LED17, LED18, LED19, LED2, LED20, LED21, LED22, LED23, LED24, LED25, LED26, LED27, LED28, LED29, LED3, LED30, LED31, LED32, LED33, LED34, LED35, LED36, LED37, LED38, LED39, LED4, LED40, LED41, LED42, LED43, LED44, LED45, LED46, LED47, LED48, LED49, LED5, LED50, LED51, LED52, LED53, LED54, LED55, LED56, LED57, LED58, LED59, LED6, LED60, LED61, LED62, LED63, LED64, LED65, LED66, LED67, LED68, LED69, LED7, LED70, LED71, LED72, LED73, LED74, LED75, LED76, LED77, LED78, LED79, LED8, LED80, LED81, LED82, LED83, LED84, LED85, LED86, LED87, LED88, LED89, LED9, LED90, LED91, LED92, LED93, LED94, LED95, LED96, LED97, LED98, LED99: QBLP677R-RGB, SamacSys_Parts:QBLP677R-RGB, symbol SamacSys_Parts:QBLP677R-RGB
Connections:
- net CS1: now also LED48.4 (COMMON_ANODE), LED64.4 (COMMON_ANODE), LED80.4 (COMMON_ANODE), LED96.4 (COMMON_ANODE)
- net CS10: now also LED105.4 (COMMON_ANODE), LED57.4 (COMMON_ANODE), LED73.4 (COMMON_ANODE), LED89.4 (COMMON_ANODE)
- net CS11: now also LED106.4 (COMMON_ANODE), LED58.4 (COMMON_ANODE), LED74.4 (COMMON_ANODE), LED90.4 (COMMON_ANODE)
- net CS12: now also LED107.4 (COMMON_ANODE), LED59.4 (COMMON_ANODE), LED75.4 (COMMON_ANODE), LED91.4 (COMMON_ANODE)
- net CS13: now also LED108.4 (COMMON_ANODE), LED60.4 (COMMON_ANODE), LED76.4 (COMMON_ANODE), LED92.4 (COMMON_ANODE)
- net CS14: now also LED109.4 (COMMON_ANODE), LED61.4 (COMMON_ANODE), LED77.4 (COMMON_ANODE), LED93.4 (COMMON_ANODE)
- net CS15: now also LED110.4 (COMMON_ANODE), LED62.4 (COMMON_ANODE), LED78.4 (COMMON_ANODE), LED94.4 (COMMON_ANODE)
- net CS16: now also LED111.4 (COMMON_ANODE), LED63.4 (COMMON_ANODE), LED79.4 (COMMON_ANODE), LED95.4 (COMMON_ANODE)
- net CS17: now also LED24.4 (COMMON_ANODE), LED8.4 (COMMON_ANODE)
- net CS18: now also LED1.4 (COMMON_ANODE), LED25.4 (COMMON_ANODE), LED9.4 (COMMON_ANODE)
- net CS19: now also LED10.4 (COMMON_ANODE), LED2.4 (COMMON_ANODE), LED26.4 (COMMON_ANODE)
- net CS2: now also LED49.4 (COMMON_ANODE), LED65.4 (COMMON_ANODE), LED81.4 (COMMON_ANODE), LED97.4 (COMMON_ANODE)
- net CS20: now also LED11.4 (COMMON_ANODE), LED27.4 (COMMON_ANODE), LED3.4 (COMMON_ANODE)
- net CS21: now also LED12.4 (COMMON_ANODE), LED28.4 (COMMON_ANODE), LED4.4 (COMMON_ANODE)
- net CS22: now also LED13.4 (COMMON_ANODE), LED29.4 (COMMON_ANODE)
- net CS23: now also LED14.4 (COMMON_ANODE), LED30.4 (COMMON_ANODE)
- net CS24: now also LED15.4 (COMMON_ANODE), LED31.4 (COMMON_ANODE)
- net CS25: now also LED16.4 (COMMON_ANODE), LED32.4 (COMMON_ANODE), LED40.4 (COMMON_ANODE)
- net CS26: now also LED17.4 (COMMON_ANODE), LED33.4 (COMMON_ANODE), LED41.4 (COMMON_ANODE)
- net CS27: now also LED18.4 (COMMON_ANODE), LED34.4 (COMMON_ANODE), LED42.4 (COMMON_ANODE)
- net CS28: now also LED19.4 (COMMON_ANODE), LED35.4 (COMMON_ANODE), LED43.4 (COMMON_ANODE)
- net CS3: now also LED50.4 (COMMON_ANODE), LED66.4 (COMMON_ANODE), LED82.4 (COMMON_ANODE), LED98.4 (COMMON_ANODE)
- net CS4: now also LED51.4 (COMMON_ANODE), LED67.4 (COMMON_ANODE), LED83.4 (COMMON_ANODE), LED99.4 (COMMON_ANODE)
- net CS5: now also LED100.4 (COMMON_ANODE), LED52.4 (COMMON_ANODE), LED68.4 (COMMON_ANODE), LED84.4 (COMMON_ANODE)
- net CS6: now also LED101.4 (COMMON_ANODE), LED53.4 (COMMON_ANODE), LED69.4 (COMMON_ANODE), LED85.4 (COMMON_ANODE)
- net CS7: now also LED102.4 (COMMON_ANODE), LED54.4 (COMMON_ANODE), LED70.4 (COMMON_ANODE), LED86.4 (COMMON_ANODE)
- net CS8: now also LED103.4 (COMMON_ANODE), LED55.4 (COMMON_ANODE), LED71.4 (COMMON_ANODE), LED87.4 (COMMON_ANODE)
- net CS9: now also LED104.4 (COMMON_ANODE), LED56.4 (COMMON_ANODE), LED72.4 (COMMON_ANODE), LED88.4 (COMMON_ANODE)
- net SW1: now also LED100.2 (CATHODE_GREEN), LED101.2 (CATHODE_GREEN), LED102.2 (CATHODE_GREEN), LED103.2 (CATHODE_GREEN), LED104.2 (CATHODE_GREEN), LED105.2 (CATHODE_GREEN), LED106.2 (CATHODE_GREEN), LED107.2 (CATHODE_GREEN), LED108.2 (CATHODE_GREEN), LED109.2 (CATHODE_GREEN), LED110.2 (CATHODE_GREEN), LED111.2 (CATHODE_GREEN), LED96.2 (CATHODE_GREEN), LED97.2 (CATHODE_GREEN), LED98.2 (CATHODE_GREEN), LED99.2 (CATHODE_GREEN)
- net SW10: now also LED48.2 (CATHODE_GREEN), LED49.2 (CATHODE_GREEN), LED50.2 (CATHODE_GREEN), LED51.2 (CATHODE_GREEN), LED52.2 (CATHODE_GREEN), LED53.2 (CATHODE_GREEN), LED54.2 (CATHODE_GREEN), LED55.2 (CATHODE_GREEN), LED56.2 (CATHODE_GREEN), LED57.2 (CATHODE_GREEN), LED58.2 (CATHODE_GREEN), LED59.2 (CATHODE_GREEN), LED60.2 (CATHODE_GREEN), LED61.2 (CATHODE_GREEN), LED62.2 (CATHODE_GREEN), LED63.2 (CATHODE_GREEN)
- net SW11: now also LED48.3 (CATHODE_RED), LED49.3 (CATHODE_RED), LED50.3 (CATHODE_RED), LED51.3 (CATHODE_RED), LED52.3 (CATHODE_RED), LED53.3 (CATHODE_RED), LED54.3 (CATHODE_RED), LED55.3 (CATHODE_RED), LED56.3 (CATHODE_RED), LED57.3 (CATHODE_RED), LED58.3 (CATHODE_RED), LED59.3 (CATHODE_RED), LED60.3 (CATHODE_RED), LED61.3 (CATHODE_RED), LED62.3 (CATHODE_RED), LED63.3 (CATHODE_RED)
- net SW12: now also LED48.1 (CATHODE_BLUE), LED49.1 (CATHODE_BLUE), LED50.1 (CATHODE_BLUE), LED51.1 (CATHODE_BLUE), LED52.1 (CATHODE_BLUE), LED53.1 (CATHODE_BLUE), LED54.1 (CATHODE_BLUE), LED55.1 (CATHODE_BLUE), LED56.1 (CATHODE_BLUE), LED57.1 (CATHODE_BLUE), LED58.1 (CATHODE_BLUE), LED59.1 (CATHODE_BLUE), LED60.1 (CATHODE_BLUE), LED61.1 (CATHODE_BLUE), LED62.1 (CATHODE_BLUE), LED63.1 (CATHODE_BLUE)
- net SW13: now also LED40.2 (CATHODE_GREEN), LED41.2 (CATHODE_GREEN), LED42.2 (CATHODE_GREEN), LED43.2 (CATHODE_GREEN), LED44.2 (CATHODE_GREEN), LED45.2 (CATHODE_GREEN), LED46.2 (CATHODE_GREEN), LED47.2 (CATHODE_GREEN)
- net SW14: now also LED40.3 (CATHODE_RED), LED41.3 (CATHODE_RED), LED42.3 (CATHODE_RED), LED43.3 (CATHODE_RED), LED44.3 (CATHODE_RED), LED45.3 (CATHODE_RED), LED46.3 (CATHODE_RED), LED47.3 (CATHODE_RED)
- net SW15: now also LED40.1 (CATHODE_BLUE), LED41.1 (CATHODE_BLUE), LED42.1 (CATHODE_BLUE), LED43.1 (CATHODE_BLUE), LED44.1 (CATHODE_BLUE), LED45.1 (CATHODE_BLUE), LED46.1 (CATHODE_BLUE), LED47.1 (CATHODE_BLUE)
- net SW16: now also LED24.2 (CATHODE_GREEN), LED25.2 (CATHODE_GREEN), LED26.2 (CATHODE_GREEN), LED27.2 (CATHODE_GREEN), LED28.2 (CATHODE_GREEN), LED29.2 (CATHODE_GREEN), LED30.2 (CATHODE_GREEN), LED31.2 (CATHODE_GREEN), LED32.2 (CATHODE_GREEN), LED33.2 (CATHODE_GREEN), LED34.2 (CATHODE_GREEN), LED35.2 (CATHODE_GREEN), LED36.2 (CATHODE_GREEN), LED37.2 (CATHODE_GREEN), LED38.2 (CATHODE_GREEN), LED39.2 (CATHODE_GREEN)
- net SW17: now also LED24.3 (CATHODE_RED), LED25.3 (CATHODE_RED), LED26.3 (CATHODE_RED), LED27.3 (CATHODE_RED), LED28.3 (CATHODE_RED), LED29.3 (CATHODE_RED), LED30.3 (CATHODE_RED), LED31.3 (CATHODE_RED), LED32.3 (CATHODE_RED), LED33.3 (CATHODE_RED), LED34.3 (CATHODE_RED), LED35.3 (CATHODE_RED), LED36.3 (CATHODE_RED), LED37.3 (CATHODE_RED), LED38.3 (CATHODE_RED), LED39.3 (CATHODE_RED)
- net SW18: now also LED24.1 (CATHODE_BLUE), LED25.1 (CATHODE_BLUE), LED26.1 (CATHODE_BLUE), LED27.1 (CATHODE_BLUE), LED28.1 (CATHODE_BLUE), LED29.1 (CATHODE_BLUE), LED30.1 (CATHODE_BLUE), LED31.1 (CATHODE_BLUE), LED32.1 (CATHODE_BLUE), LED33.1 (CATHODE_BLUE), LED34.1 (CATHODE_BLUE), LED35.1 (CATHODE_BLUE), LED36.1 (CATHODE_BLUE), LED37.1 (CATHODE_BLUE), LED38.1 (CATHODE_BLUE), LED39.1 (CATHODE_BLUE)
- net SW19: now also LED10.2 (CATHODE_GREEN), LED11.2 (CATHODE_GREEN), LED12.2 (CATHODE_GREEN), LED13.2 (CATHODE_GREEN), LED14.2 (CATHODE_GREEN), LED15.2 (CATHODE_GREEN), LED16.2 (CATHODE_GREEN), LED17.2 (CATHODE_GREEN), LED18.2 (CATHODE_GREEN), LED19.2 (CATHODE_GREEN), LED20.2 (CATHODE_GREEN), LED21.2 (CATHODE_GREEN), LED22.2 (CATHODE_GREEN), LED23.2 (CATHODE_GREEN), LED8.2 (CATHODE_GREEN), LED9.2 (CATHODE_GREEN)
- net SW2: now also LED100.3 (CATHODE_RED), LED101.3 (CATHODE_RED), LED102.3 (CATHODE_RED), LED103.3 (CATHODE_RED), LED104.3 (CATHODE_RED), LED105.3 (CATHODE_RED), LED106.3 (CATHODE_RED), LED107.3 (CATHODE_RED), LED108.3 (CATHODE_RED), LED109.3 (CATHODE_RED), LED110.3 (CATHODE_RED), LED111.3 (CATHODE_RED), LED96.3 (CATHODE_RED), LED97.3 (CATHODE_RED), LED98.3 (CATHODE_RED), LED99.3 (CATHODE_RED)
- net SW20: now also LED10.3 (CATHODE_RED), LED11.3 (CATHODE_RED), LED12.3 (CATHODE_RED), LED13.3 (CATHODE_RED), LED14.3 (CATHODE_RED), LED15.3 (CATHODE_RED), LED16.3 (CATHODE_RED), LED17.3 (CATHODE_RED), LED18.3 (CATHODE_RED), LED19.3 (CATHODE_RED), LED20.3 (CATHODE_RED), LED21.3 (CATHODE_RED), LED22.3 (CATHODE_RED), LED23.3 (CATHODE_RED), LED8.3 (CATHODE_RED), LED9.3 (CATHODE_RED)
- net SW21: now also LED10.1 (CATHODE_BLUE), LED11.1 (CATHODE_BLUE), LED12.1 (CATHODE_BLUE), LED13.1 (CATHODE_BLUE), LED14.1 (CATHODE_BLUE), LED15.1 (CATHODE_BLUE), LED16.1 (CATHODE_BLUE), LED17.1 (CATHODE_BLUE), LED18.1 (CATHODE_BLUE), LED19.1 (CATHODE_BLUE), LED20.1 (CATHODE_BLUE), LED21.1 (CATHODE_BLUE), LED22.1 (CATHODE_BLUE), LED23.1 (CATHODE_BLUE), LED8.1 (CATHODE_BLUE), LED9.1 (CATHODE_BLUE)
- net SW22: now also LED1.2 (CATHODE_GREEN), LED2.2 (CATHODE_GREEN), LED3.2 (CATHODE_GREEN), LED4.2 (CATHODE_GREEN), LED5.2 (CATHODE_GREEN), LED6.2 (CATHODE_GREEN), LED7.2 (CATHODE_GREEN)
- net SW23: now also LED1.3 (CATHODE_RED), LED2.3 (CATHODE_RED), LED3.3 (CATHODE_RED), LED4.3 (CATHODE_RED), LED5.3 (CATHODE_RED), LED6.3 (CATHODE_RED), LED7.3 (CATHODE_RED)
- net SW24: now also LED1.1 (CATHODE_BLUE), LED2.1 (CATHODE_BLUE), LED3.1 (CATHODE_BLUE), LED4.1 (CATHODE_BLUE), LED5.1 (CATHODE_BLUE), LED6.1 (CATHODE_BLUE), LED7.1 (CATHODE_BLUE)
- net SW3: now also LED100.1 (CATHODE_BLUE), LED101.1 (CATHODE_BLUE), LED102.1 (CATHODE_BLUE), LED103.1 (CATHODE_BLUE), LED104.1 (CATHODE_BLUE), LED105.1 (CATHODE_BLUE), LED106.1 (CATHODE_BLUE), LED107.1 (CATHODE_BLUE), LED108.1 (CATHODE_BLUE), LED109.1 (CATHODE_BLUE), LED110.1 (CATHODE_BLUE), LED111.1 (CATHODE_BLUE), LED96.1 (CATHODE_BLUE), LED97.1 (CATHODE_BLUE), LED98.1 (CATHODE_BLUE), LED99.1 (CATHODE_BLUE)
- net SW4: now also LED80.2 (CATHODE_GREEN), LED81.2 (CATHODE_GREEN), LED82.2 (CATHODE_GREEN), LED83.2 (CATHODE_GREEN), LED84.2 (CATHODE_GREEN), LED85.2 (CATHODE_GREEN), LED86.2 (CATHODE_GREEN), LED87.2 (CATHODE_GREEN), LED88.2 (CATHODE_GREEN), LED89.2 (CATHODE_GREEN), LED90.2 (CATHODE_GREEN), LED91.2 (CATHODE_GREEN), LED92.2 (CATHODE_GREEN), LED93.2 (CATHODE_GREEN), LED94.2 (CATHODE_GREEN), LED95.2 (CATHODE_GREEN)
- net SW5: now also LED80.3 (CATHODE_RED), LED81.3 (CATHODE_RED), LED82.3 (CATHODE_RED), LED83.3 (CATHODE_RED), LED84.3 (CATHODE_RED), LED85.3 (CATHODE_RED), LED86.3 (CATHODE_RED), LED87.3 (CATHODE_RED), LED88.3 (CATHODE_RED), LED89.3 (CATHODE_RED), LED90.3 (CATHODE_RED), LED91.3 (CATHODE_RED), LED92.3 (CATHODE_RED), LED93.3 (CATHODE_RED), LED94.3 (CATHODE_RED), LED95.3 (CATHODE_RED)
- net SW6: now also LED80.1 (CATHODE_BLUE), LED81.1 (CATHODE_BLUE), LED82.1 (CATHODE_BLUE), LED83.1 (CATHODE_BLUE), LED84.1 (CATHODE_BLUE), LED85.1 (CATHODE_BLUE), LED86.1 (CATHODE_BLUE), LED87.1 (CATHODE_BLUE), LED88.1 (CATHODE_BLUE), LED89.1 (CATHODE_BLUE), LED90.1 (CATHODE_BLUE), LED91.1 (CATHODE_BLUE), LED92.1 (CATHODE_BLUE), LED93.1 (CATHODE_BLUE), LED94.1 (CATHODE_BLUE), LED95.1 (CATHODE_BLUE)
- net SW7: now also LED64.2 (CATHODE_GREEN), LED65.2 (CATHODE_GREEN), LED66.2 (CATHODE_GREEN), LED67.2 (CATHODE_GREEN), LED68.2 (CATHODE_GREEN), LED69.2 (CATHODE_GREEN), LED70.2 (CATHODE_GREEN), LED71.2 (CATHODE_GREEN), LED72.2 (CATHODE_GREEN), LED73.2 (CATHODE_GREEN), LED74.2 (CATHODE_GREEN), LED75.2 (CATHODE_GREEN), LED76.2 (CATHODE_GREEN), LED77.2 (CATHODE_GREEN), LED78.2 (CATHODE_GREEN), LED79.2 (CATHODE_GREEN)
- net SW8: now also LED64.3 (CATHODE_RED), LED65.3 (CATHODE_RED), LED66.3 (CATHODE_RED), LED67.3 (CATHODE_RED), LED68.3 (CATHODE_RED), LED69.3 (CATHODE_RED), LED70.3 (CATHODE_RED), LED71.3 (CATHODE_RED), LED72.3 (CATHODE_RED), LED73.3 (CATHODE_RED), LED74.3 (CATHODE_RED), LED75.3 (CATHODE_RED), LED76.3 (CATHODE_RED), LED77.3 (CATHODE_RED), LED78.3 (CATHODE_RED), LED79.3 (CATHODE_RED)
- net SW9: now also LED64.1 (CATHODE_BLUE), LED65.1 (CATHODE_BLUE), LED66.1 (CATHODE_BLUE), LED67.1 (CATHODE_BLUE), LED68.1 (CATHODE_BLUE), LED69.1 (CATHODE_BLUE), LED70.1 (CATHODE_BLUE), LED71.1 (CATHODE_BLUE), LED72.1 (CATHODE_BLUE), LED73.1 (CATHODE_BLUE), LED74.1 (CATHODE_BLUE), LED75.1 (CATHODE_BLUE), LED76.1 (CATHODE_BLUE), LED77.1 (CATHODE_BLUE), LED78.1 (CATHODE_BLUE), LED79.1 (CATHODE_BLUE)
- new net CS29: LED20.4 (COMMON_ANODE), LED36.4 (COMMON_ANODE), LED44.4 (COMMON_ANODE)
- new net CS30: LED21.4 (COMMON_ANODE), LED37.4 (COMMON_ANODE), LED45.4 (COMMON_ANODE), LED5.4 (COMMON_ANODE)
- new net CS31: LED22.4 (COMMON_ANODE), LED38.4 (COMMON_ANODE), LED46.4 (COMMON_ANODE), LED6.4 (COMMON_ANODE)
- new net CS32: LED23.4 (COMMON_ANODE), LED39.4 (COMMON_ANODE), LED47.4 (COMMON_ANODE), LED7.4 (COMMON_ANODE)
