File: TooManyKeys/KiCad/TooManyKeys.kicad_pcb (KiCad board)
At the start: 2 copper layers, 430.2 x 141.3 mm, 394 parts, among them J1 54104-3031_Oled, J2 AVR-ISP-6, SW1 SW_Push, U1 PRTR5V0U2X, U2 AT90USB1286-AU, U3 PCA9306, U4 AZ1117CH-3.3TRG1, Y1 16MHz

Commit message: Flip Led Footprint
Added version 1.5 to pcb
Added version 1.2 to sch
Added proper Level Shifter to BOM
Routing:
- net SW18: track 475.8 -> 457.1 mm
- net SW21: track 536.4 -> 520.1 mm
- net SW24: track 357.6 -> 346.1 mm, vias 15 -> 14
- net CS27: track 361.2 -> 371.5 mm
- net CS31: track 280.4 -> 283.1 mm
- net CS32: track 249.9 -> 252.5 mm
- net CS26: track 356.8 -> 359.1 mm
- net CS23: track 191.9 -> 190.4 mm
- net CS17: track 294.3 -> 292.8 mm
- net CS24: track 144.7 -> 143.3 mm
- net CS19: track 268.6 -> 267.5 mm
- net CS21: track 236.0 -> 236.6 mm
Other:
- board text added: "TooManyKeys V1.5"
- board text removed: "TooManyKeys V1.0"

Commit message: Finished work on new led footprint, need to double check
Parts:
- removed MX_RSFT1: MX-NoLED, MX_Only:MXOnly-2.75U-NoLED_3Pins
Routing:
- net SW6: track 727.6 -> 695.9 mm, vias 37 -> 35
- net SW9: track 614.1 -> 593.1 mm, vias 36 -> 33
- net SW15: track 357.0 -> 339.2 mm
- net SW12: track 507.1 -> 491.5 mm
- net CS12: track 364.9 -> 353.5 mm
- net SW3: track 807.5 -> 797.3 mm, vias 33 -> 32
- net CS15: track 381.0 -> 389.3 mm, vias 10 -> 12
- net CS16: track 439.4 -> 444.9 mm, vias 10 -> 9
- net CS26: track 359.1 -> 364.3 mm
- net CS31: track 283.1 -> 288.1 mm
- net CS10: track 309.2 -> 313.3 mm
- net CS9: track 280.8 -> 284.9 mm
- net CS4: track 272.5 -> 275.7 mm
- net CS6: track 299.0 -> 302.1 mm
- net CS27: track 371.5 -> 374.6 mm
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
Commit message: Set Led footprint text position
Renaming items in footprint library
Parts:
- U3: footprint SamacSys_Parts:SOP50P310X90-8N -> SamacSys_Parts:PCA9306TDCURQ1
Routing:
- net Net-(D93-Pad2): track 6.82 -> 0.00 mm
- net GND: vias 93 -> 91

Commit message: Updating pcb with IS31FL3733-TQLS4 footprint
Parts:
- MASTER_U1, SLAVE_U1: footprint SamacSys_Parts:QFP50P900X900X120-49N -> SamacSys_Parts:IS31FL3733-TQLS4
