File: TooManyKeys/KiCad/TooManyKeys.kicad_pcb (KiCad board)
At the start: 2 copper layers, 430.2 x 141.3 mm, 394 parts, among them J1 54104-3031_Oled, J2 AVR-ISP-6, SW1 SW_Push, U1 PRTR5V0U2X, U2 AT90USB1286-AU, U3 PCA9306TDCURQ1, U4 AZ1117CH-3.3TRG1, Y1 16MHz

Commit message: Final routing + properly saved 3 pins footprint
Parts:
- MX_0, MX_1, MX_2, MX_3, MX_4, MX_5, MX_6, MX_7, MX_8, MX_9, MX_A1, MX_B1, MX_C1, MX_COMM1, MX_D1, MX_DEL1, MX_DOT1, MX_DOWN1, MX_E1, MX_END1, MX_EQL1, MX_ESC1, MX_F1, MX_F11, MX_F12, MX_F13, MX_F2, MX_F3, MX_F4, MX_F5, MX_F6, MX_F7, MX_F8, MX_F9, MX_G1, MX_GRV1, MX_H1, MX_HOME1, MX_I1, MX_INS1, MX_J1, MX_K1, MX_L1, MX_LBRC1, MX_LEFT1, MX_M1, MX_MINS1, MX_MUTE1, MX_N1, MX_NEXT1, MX_NLCK1, MX_O1, MX_P*1, MX_P-1, MX_P/1, MX_P1, MX_P10, MX_P2, MX_P3, MX_P4, MX_P5, MX_P6, MX_P7, MX_P8, MX_P9, MX_PAUSE1, MX_PDOT1, MX_PGDN1, MX_PGUP1, MX_PLAY1, MX_PREV1, MX_PSCR1, MX_Q1, MX_QUOT1, MX_R1, MX_RBRC1, MX_RGHT1, MX_S1, MX_SCLN1, MX_SLCK1, MX_SLSH1, MX_STOP1, MX_T1, MX_U1, MX_UP1, MX_V1, MX_VOLD1, MX_VOLU1, MX_W1, MX_X1, MX_Y1, MX_Z1: footprint MX_Only:MXOnly-1U-NoLED_3Pins -> SamacSys_Parts:MXOnly-1U-NoLED_3Pins
- MX_RSFT1: footprint MX_Only:MXOnly-2.75U-NoLED -> SamacSys_Parts:MXOnly-2.75U-NoLED_3Pins
Routing:
- net SW16: track 455.2 -> 447.4 mm
- net SW19: track 472.1 -> 465.1 mm
- net SW10: track 639.9 -> 636.5 mm
- net SW13: track 304.0 -> 300.9 mm
- net (no net): track 2.02 -> 0.00 mm
- net SW22: track 327.5 -> 325.5 mm
- net SW7: track 576.1 -> 574.9 mm
- net SW8: track 635.8 -> 635.2 mm
